File: Housekeeping.kicad_sch (KiCad schematic)
At the start: 46 parts

Commit message: Updated Schmatics
Some outdated schematics were in the init commit. Uploded proper revision with tweaks.
Parts:
- removed C? (x10): 100nF, symbol Device:C_Small
- removed C? (x9): 150pF, symbol Device:C_Small
- removed C?: 220pF, symbol Device:C_Small
- removed D?: Green, symbol Device:LED
- removed J? (x2): Conn_02x10_Odd_Even, symbol Connector_Generic:Conn_02x10_Odd_Even
- removed R? (x5): 22k, symbol Device:R_Small_US
- removed R? (x11): 4.75k, symbol Device:R_Small_US
- removed R?: 150R, symbol Device:R_Small_US
- removed U? (x3): ~, symbol Custom_Lib_MPEX_Zest:74LVC8T245
- removed U?: AMC7823IRTAR, QFN50P600X600X80-41N, symbol AMC7823IRTAR:AMC7823IRTAR
- removed U? (x2): ~, symbol Custom_Lib_MPEX_Zest:74LVC4T245
- added C? (x9): 150pF, symbol Device:C_Small
- added C? (x14): 100nF, symbol Device:C_Small
- added C? (x8): 100nF, Capacitor_SMD:C_0603_1608Metric, symbol Device:C_Small
- added C?: 220pF, symbol Device:C_Small
- added D?: Green, symbol Device:LED
- added J? (x2): Conn_02x10_Odd_Even, symbol Connector_Generic:Conn_02x10_Odd_Even
- added R? (x5): 22k, symbol Device:R_Small_US
- added R? (x9): 4.75k, symbol Device:R_Small_US
- added R?: 150R, symbol Device:R_Small_US
- added U123 (x8): MAX4896, symbol AD7768_Digitizer_SLib:MAX4896
- added U? (x7): 74LVC8T245, symbol Custom_Lib_MPEX_Zest:74LVC8T245
- added U?: AMC7823IRTAR, QFN50P600X600X80-41N, symbol AMC7823IRTAR:AMC7823IRTAR
Connections:
- net AD0: now also C?.1, J?.9 (Pin_9), U?.11 (CH0)
- net AD1: now also C?.1, J?.7 (Pin_7), U?.12 (CH1)
- net AD2: now also C?.1, J?.5 (Pin_5), U?.13 (CH2)
- net AD3: now also C?.1, J?.3 (Pin_3), U?.14 (CH3)
- net AD4: now also C?.1, J?.1 (Pin_1), U?.17 (CH4)
- net AD5: now also U?.18 (CH5)
- net AD7: now also R?.1, R?.2, U?.20 (CH7)
- net AMC7823_SPI_MISO: now also U?.18 (B4), U?.34 (MISO)
- net AMC7823_SPI_SS: now also U?.21 (B1), U?.35 (~{SS})
- net DAC0: now also J?.17 (Pin_17), U?.6 (DAC0_OUT)
- net DAC1: now also J?.15 (Pin_15), U?.7 (DAC1_OUT)
- net DAC2: now also J?.13 (Pin_13), U?.8 (DAC2_OUT)
- net DAC3: now also J?.11 (Pin_11), U?.9 (DAC3_OUT)
- net DAC4: now also J?.17 (Pin_17), U?.22 (DAC4_OUT)
- net DAC5: now also J?.15 (Pin_15), U?.23 (DAC5_OUT)
- net DAC6: now also J?.13 (Pin_13), U?.24 (DAC6_OUT)
- net DAC7: now also J?.11 (Pin_11), U?.25 (DAC7_OUT)
- net EXT_REFIN: now also J?.19 (Pin_19), U?.21 (EXT_REF_IN)
- net GND: now also C?.1, C?.1, C?.1, C?.1, C?.1, C?.1, C?.1, C?.1, C?.1, C?.1, C?.1, C?.1, C?.1, C?.1, C?.1, C?.1, C?.1, C?.1, C?.2, C?.2, C?.2, C?.2, C?.2, C?.2, C?.2, C?.2, C?.2, C?.2, C?.2, C?.2, C?.2, C?.2, J?.10 (Pin_10), J?.10 (Pin_10), J?.12 (Pin_12), J?.12 (Pin_12), J?.14 (Pin_14), J?.14 (Pin_14), J?.16 (Pin_16), J?.16 (Pin_16), J?.18 (Pin_18), J?.18 (Pin_18), J?.2 (Pin_2), J?.2 (Pin_2), J?.20 (Pin_20), J?.20 (Pin_20), J?.4 (Pin_4), J?.4 (Pin_4), J?.6 (Pin_6), J?.6 (Pin_6), J?.8 (Pin_8), J?.8 (Pin_8), R?.2, R?.2, U123.10 (PGND), U123.10 (PGND), U123.10 (PGND), U123.10 (PGND), U123.10 (PGND), U123.10 (PGND), U123.10 (PGND), U123.10 (PGND), U123.13 (GND), U123.13 (GND), U123.13 (GND), U123.13 (GND), U123.13 (GND), U123.13 (GND), U123.13 (GND), U123.13 (GND), U123.21 (EP), U123.21 (EP), U123.21 (EP), U123.21 (EP), U123.21 (EP), U123.21 (EP), U123.21 (EP), U123.21 (EP), U123.6 (PDCD), U123.6 (PDCD), U123.6 (PDCD), U123.6 (PDCD), U123.6 (PDCD), U123.6 (PDCD), U123.6 (PDCD), U123.6 (PDCD), U123.7 (SPLD), U123.7 (SPLD), U123.7 (SPLD), U123.7 (SPLD), U123.7 (SPLD), U123.7 (SPLD), U123.7 (SPLD), U123.7 (SPLD), U?.10 (SGND), U?.11 (GND), U?.11 (GND), U?.11 (GND), U?.11 (GND), U?.11 (GND), U?.11 (GND), U?.11 (GND), U?.12 (GND), U?.12 (GND), U?.12 (GND), U?.12 (GND), U?.12 (GND), U?.12 (GND), U?.12 (GND), U?.13 (GND), U?.13 (GND), U?.13 (GND), U?.13 (GND), U?.13 (GND), U?.13 (GND), U?.13 (GND), U?.15 (AGND), U?.2 (DIR), U?.2 (DIR), U?.2 (DIR), U?.22 (OE), U?.22 (OE), U?.22 (OE), U?.22 (OE), U?.22 (OE), U?.22 (OE), U?.22 (OE), U?.38 (DGND), U?.41 (EXP)
- net GPIO0: now also J?.9 (Pin_9), R?.2, U?.27 (GPIO-0/~{ALR0})
- net GPIO1: now also J?.7 (Pin_7), R?.2, U?.28 (GPIO-1/~{ALR1})
- net GPIO2: now also J?.5 (Pin_5), R?.2, U?.29 (GPIO-2/~{ALR2})
- net GPIO3: now also J?.3 (Pin_3), R?.2, U?.30 (GPIO-3/~{ALR3})
- net GPIO4: now also R?.2, U?.39 (GPIO-4)
- net GPIO5: now also R?.1, U?.40 (GPIO-5)
- net I_MON: now also C?.1, U?.19 (CH6)
- net P2_ADC_SCLK: now also U?.3 (A1)
- net P2_AMC7823_SPI_MISO: now also U?.6 (A4)
- net P2_AMC7823_SPI_SS: now also U?.3 (A1)
- net P2_POLL_MOSI: now also U?.5 (A3)
- net P2_POLL_SCLK: now also U?.4 (A2)
- net P2_VADJ: now also C?.2, C?.2, C?.2, C?.2, C?.2, C?.2, C?.2, R?.2, R?.2, R?.2, R?.2, U?.1 (VCCA), U?.1 (VCCA), U?.1 (VCCA), U?.1 (VCCA), U?.1 (VCCA), U?.1 (VCCA), U?.1 (VCCA)
- net VDD1P8V: now also C?.2, C?.2, C?.2, C?.2, C?.2, U?.23 (VCCB), U?.23 (VCCB), U?.23 (VCCB), U?.23 (VCCB), U?.23 (VCCB), U?.24 (VCCB), U?.24 (VCCB), U?.24 (VCCB), U?.24 (VCCB), U?.24 (VCCB)
- net VDD3P3V: now also C?.2, C?.2, C?.2, C?.2, C?.2, C?.2, D?.2 (A), R?.1, R?.1, R?.1, R?.1, R?.1, R?.1, R?.1, R?.2, U?.16 (AVDD), U?.23 (VCCB), U?.23 (VCCB), U?.24 (VCCB), U?.24 (VCCB), U?.36 (BVDD), U?.37 (DVDD)
- new net: D?.1 (K), R?.2
- new net: J?.19 (Pin_19), U?.5 (PRECISION_I_OUTPUT)
- new net: R?.1, U?.26 (~{RESET})
- new net: J?.1 (Pin_1), U?.31 (CONVERT)
- new net: R?.2, U?.4 (ISET_RESISTOR)
- new net: R?.1, U?.2 (DIR) (x4)
- new net: R?.1, U?.3 (ELDAC)
- new net: U123.3 (DIN), U123.5 (DOUT) (x7)
- new net +5V: C?.1, C?.1, C?.1, C?.1, C?.1, C?.1, C?.1, C?.1, U123.1 (~{RESET}), U123.1 (~{RESET}), U123.1 (~{RESET}), U123.1 (~{RESET}), U123.1 (~{RESET}), U123.1 (~{RESET}), U123.1 (~{RESET}), U123.1 (~{RESET})
- new net AD7768_Filter: U?.19 (B3)
- new net AD7768_Mode_0: U?.15 (B7)
- new net AD7768_Mode_1: U?.16 (B6)
- new net AD7768_Mode_2: U?.17 (B5)
- new net AD7768_Mode_3: U?.18 (B4)
- new net AD7768_SCLK: U?.21 (B1)
- new net AD7768_~{RESET}: U?.20 (B2)
- new net AD7768_~{Start}: U?.21 (B1)
- new net AD7768_~{Sync_In}: U?.20 (B2)
- new net AD7768_~{Sync_Out}: U?.21 (B1)
- new net ADC1_DCLK: U?.19 (B3)
- new net ADC1_SDI: U?.17 (B5)
- new net ADC1_SDO: U?.17 (B5)
- new net ADC1_~{CS}: U?.21 (B1)
- new net ADC1_~{DRDY}: U?.21 (B1)
- new net ADC2_DCLK: U?.18 (B4)
- new net ADC2_SDI: U?.16 (B6)
- new net ADC2_SDO: U?.16 (B6)
- new net ADC2_~{CS}: U?.20 (B2)
- new net ADC2_~{DRDY}: U?.20 (B2)
- new net ADC3_DCLK: U?.17 (B5)
- new net ADC3_SDI: U?.15 (B7)
- new net ADC3_SDO: U?.15 (B7)
- new net ADC3_~{CS}: U?.19 (B3)
- new net ADC3_~{DRDY}: U?.19 (B3)
- new net ADC4_DCLK: U?.16 (B6)
- new net ADC4_SDI: U?.14 (B8)
- new net ADC4_SDO: U?.14 (B8)
- new net ADC4_~{CS}: U?.18 (B4)
- new net ADC4_~{DRDY}: U?.18 (B4)
- new net AMC7823_SPI_MOSI: U?.19 (B3), U?.33 (MOSI)
- new net AMC7823_SPI_SCLK: U?.20 (B2), U?.32 (SCLK)
- new net MAX4896_Reset: U123.1 (~{RESET}), U123.1 (~{RESET}), U123.1 (~{RESET}), U123.1 (~{RESET}), U123.1 (~{RESET}), U123.1 (~{RESET}), U123.1 (~{RESET}), U123.1 (~{RESET}), U?.17 (B5)
- new net MAX4896_SCLK: U123.4 (SCLK), U123.4 (SCLK), U123.4 (SCLK), U123.4 (SCLK), U123.4 (SCLK), U123.4 (SCLK), U123.4 (SCLK), U123.4 (SCLK), U?.16 (B6)
- new net MAX4896_~{CS}: U123.2 (~{CS}), U123.2 (~{CS}), U123.2 (~{CS}), U123.2 (~{CS}), U123.2 (~{CS}), U123.2 (~{CS}), U123.2 (~{CS}), U123.2 (~{CS}), U?.15 (B7)
- new net MAX4896_~{FLAG}1: U123.15 (~{FLAG}), U?.21 (B1)
- new net MAX4896_~{FLAG}2: U123.15 (~{FLAG}), U?.20 (B2)
- new net MAX4896_~{FLAG}3: U123.15 (~{FLAG}), U?.19 (B3)
- new net MAX4896_~{FLAG}4: U123.15 (~{FLAG}), U?.18 (B4)
- new net MAX4896_~{FLAG}5: U123.15 (~{FLAG}), U?.17 (B5)
- new net MAX4896_~{FLAG}6: U123.15 (~{FLAG}), U?.16 (B6)
- new net MAX4896_~{FLAG}7: U123.15 (~{FLAG}), U?.15 (B7)
- new net MAX4896_~{FLAG}8: U123.15 (~{FLAG}), U?.14 (B8)
- new net P2_ADC1_DCLK: U?.5 (A3)
- new net P2_ADC1_SDI: U?.7 (A5)
- new net P2_ADC1_SDO: U?.7 (A5)
- new net P2_ADC1_~{CS}: U?.3 (A1)
- new net P2_ADC1_~{DRDY}: U?.3 (A1)
- new net P2_ADC2_DCLK: U?.6 (A4)
- new net P2_ADC2_SDI: U?.8 (A6)
- new net P2_ADC2_SDO: U?.8 (A6)
- new net P2_ADC2_~{CS}: U?.4 (A2)
- new net P2_ADC2_~{DRDY}: U?.4 (A2)
- new net P2_ADC3_DCLK: U?.7 (A5)
- new net P2_ADC3_SDI: U?.9 (A7)
- new net P2_ADC3_SDO: U?.9 (A7)
- new net P2_ADC3_~{CS}: U?.5 (A3)
- new net P2_ADC3_~{DRDY}: U?.5 (A3)
- new net P2_ADC4_DCLK: U?.8 (A6)
- new net P2_ADC4_SDI: U?.10 (A8)
- new net P2_ADC4_SDO: U?.10 (A8)
- new net P2_ADC4_~{CS}: U?.6 (A4)
- new net P2_ADC4_~{DRDY}: U?.6 (A4)
- new net P2_ADC_Filter: U?.5 (A3)
- new net P2_ADC_Mode_0: U?.9 (A7)
- new net P2_ADC_Mode_1: U?.8 (A6)
- new net P2_ADC_Mode_2: U?.7 (A5)
- new net P2_ADC_Mode_3: U?.6 (A4)
- new net P2_ADC_~{RESET}: U?.4 (A2)
- new net P2_ADC_~{Start}: U?.3 (A1)
- new net P2_ADC_~{Sync_In}: U?.4 (A2)
- new net P2_ADC_~{Sync_Out}: U?.3 (A1)
- new net P2_MAX4896_Reset: U?.7 (A5)
- new net P2_MAX4896_SCLK: U?.8 (A6)
- new net P2_MAX4896_~{CS}: U?.9 (A7)
- new net P2_MAX4896_~{FLAG}1: U?.3 (A1)
- new net P2_MAX4896_~{FLAG}2: U?.4 (A2)
- new net P2_MAX4896_~{FLAG}3: U?.5 (A3)
- new net P2_MAX4896_~{FLAG}4: U?.6 (A4)
- new net P2_MAX4896_~{FLAG}5: U?.7 (A5)
- new net P2_MAX4896_~{FLAG}6: U?.8 (A6)
- new net P2_MAX4896_~{FLAG}7: U?.9 (A7)
- new net P2_MAX4896_~{FLAG}8: U?.10 (A8)
- new net P2_Relay_ShiftData: U?.10 (A8)
- new net PGND: U123.16 (PGND), U123.16 (PGND), U123.16 (PGND), U123.16 (PGND), U123.16 (PGND), U123.16 (PGND), U123.16 (PGND), U123.16 (PGND)
- new net Relay_ResetCoil1: U123.18 (OUT1)
- new net Relay_ResetCoil10: U123.17 (OUT2)
- new net Relay_ResetCoil11: U123.15 (~{FLAG})
- new net Relay_ResetCoil12: U123.14 (OUT4)
- new net Relay_ResetCoil13: U123.12 (OUT5)
- new net Relay_ResetCoil14: U123.11 (OUT6)
- new net Relay_ResetCoil15: U123.9 (OUT7)
- new net Relay_ResetCoil16: U123.8 (OUT8)
- new net Relay_ResetCoil17: U123.18 (OUT1)
- new net Relay_ResetCoil18: U123.17 (OUT2)
- new net Relay_ResetCoil19: U123.15 (~{FLAG})
- new net Relay_ResetCoil2: U123.17 (OUT2)
- new net Relay_ResetCoil20: U123.14 (OUT4)
- new net Relay_ResetCoil21: U123.12 (OUT5)
- new net Relay_ResetCoil22: U123.11 (OUT6)
- new net Relay_ResetCoil23: U123.9 (OUT7)
- new net Relay_ResetCoil24: U123.8 (OUT8)
- new net Relay_ResetCoil25: U123.18 (OUT1)
- new net Relay_ResetCoil26: U123.17 (OUT2)
- new net Relay_ResetCoil27: U123.15 (~{FLAG})
- new net Relay_ResetCoil28: U123.14 (OUT4)
- new net Relay_ResetCoil29: U123.12 (OUT5)
- new net Relay_ResetCoil3: U123.15 (~{FLAG})
- new net Relay_ResetCoil30: U123.11 (OUT6)
- new net Relay_ResetCoil31: U123.9 (OUT7)
- new net Relay_ResetCoil32: U123.8 (OUT8)
- new net Relay_ResetCoil4: U123.14 (OUT4)
- new net Relay_ResetCoil5: U123.12 (OUT5)
- new net Relay_ResetCoil6: U123.11 (OUT6)
- new net Relay_ResetCoil7: U123.9 (OUT7)
- new net Relay_ResetCoil8: U123.8 (OUT8)
- new net Relay_ResetCoil9: U123.18 (OUT1)
- new net Relay_SetCoil1: U123.18 (OUT1)
- new net Relay_SetCoil10: U123.17 (OUT2)
- new net Relay_SetCoil11: U123.15 (~{FLAG})
- new net Relay_SetCoil12: U123.14 (OUT4)
- new net Relay_SetCoil13: U123.12 (OUT5)
- new net Relay_SetCoil14: U123.11 (OUT6)
- new net Relay_SetCoil15: U123.9 (OUT7)
- new net Relay_SetCoil16: U123.8 (OUT8)
- new net Relay_SetCoil17: U123.18 (OUT1)
- new net Relay_SetCoil18: U123.17 (OUT2)
- new net Relay_SetCoil19: U123.15 (~{FLAG})
- new net Relay_SetCoil2: U123.17 (OUT2)
- new net Relay_SetCoil20: U123.14 (OUT4)
- new net Relay_SetCoil21: U123.12 (OUT5)
- new net Relay_SetCoil22: U123.11 (OUT6)
- new net Relay_SetCoil23: U123.9 (OUT7)
- new net Relay_SetCoil24: U123.8 (OUT8)
- new net Relay_SetCoil25: U123.18 (OUT1)
- new net Relay_SetCoil26: U123.17 (OUT2)
- new net Relay_SetCoil27: U123.15 (~{FLAG})
- new net Relay_SetCoil28: U123.14 (OUT4)
- new net Relay_SetCoil29: U123.12 (OUT5)
- new net Relay_SetCoil3: U123.15 (~{FLAG})
- new net Relay_SetCoil30: U123.11 (OUT6)
- new net Relay_SetCoil31: U123.9 (OUT7)
- new net Relay_SetCoil32: U123.8 (OUT8)
- new net Relay_SetCoil4: U123.14 (OUT4)
- new net Relay_SetCoil5: U123.12 (OUT5)
- new net Relay_SetCoil6: U123.11 (OUT6)
- new net Relay_SetCoil7: U123.9 (OUT7)
- new net Relay_SetCoil8: U123.8 (OUT8)
- new net Relay_SetCoil9: U123.18 (OUT1)
- new net Relay_ShiftData: U123.3 (DIN), U?.14 (B8)

Commit message: Fixed FMC mapping Issue
Fixed FMC pin mapping and added FMC pin mapping excel file
Parts:
- added C? (x2): 1uF, Capacitor_SMD:C_0603_1608Metric, symbol Device:C_Small
- added C? (x2): 100nF, symbol Device:C_Small
- added R? (x3): 0R, symbol Device:R_Small_US
- added R?: 11.5k, symbol Device:R_Small_US
- added R? (x3): 4.75k, symbol Device:R_Small_US
- added U14: AD7794, Package_SO:TSSOP-24_4.4x7.8mm_P0.65mm, symbol Analog_ADC:AD7794
- added U15: AT24C64D-SSHM, Package_SO:SOIC-8_3.9x4.9mm_P1.27mm, symbol Memory_EEPROM:AT24CS01-SSHM
- added U?: 74LVC8T245, symbol Custom_Lib_MPEX_Zest:74LVC8T245
Connections:
- net AMC7823_SPI_MOSI: now also U14.24 (DIN)
- net AMC7823_SPI_SCLK: now also U14.1 (SCLK)
- net GND: now also C?.1, C?.1, C?.2, C?.2, R?.1, R?.2, U14.20 (GND), U15.3 (A2), U15.4 (GND), U?.11 (GND), U?.12 (GND), U?.13 (GND), U?.22 (OE)
- net P2_VADJ: now also C?.2, R?.2, U?.1 (VCCA)
- net VDD3P3V: now also C?.2, U?.23 (VCCB), U?.24 (VCCB)
- net P2_ADC1_DCLK renamed P1_ADC1_DCLK
- net P2_ADC1_SDI renamed P1_ADC1_SDI
- net P2_ADC1_SDO renamed P1_ADC1_SDO
- net P2_ADC1_~{CS} renamed P1_ADC1_~{CS}
- net P2_ADC1_~{DRDY} renamed P1_ADC1_~{DRDY}
- net P2_ADC2_DCLK renamed P1_ADC2_DCLK
- net P2_ADC2_SDI renamed P1_ADC2_SDI
- net P2_ADC2_SDO renamed P1_ADC2_SDO
- net P2_ADC2_~{CS} renamed P1_ADC2_~{CS}
- net P2_ADC2_~{DRDY} renamed P1_ADC2_~{DRDY}
- net P2_ADC_Filter renamed P1_ADC_Filter
- net P2_ADC_Mode_0 renamed P1_ADC_Mode_0
- net P2_ADC_Mode_1 renamed P1_ADC_Mode_1
- net P2_ADC_Mode_2 renamed P1_ADC_Mode_2
- net P2_ADC_Mode_3 renamed P1_ADC_Mode_3
- net P2_ADC_SCLK renamed P1_ADC_SCLK
- net P2_ADC_~{RESET} renamed P1_ADC_~{RESET}
- net P2_ADC_~{Start} renamed P1_ADC_~{Start}
- net P2_ADC_~{Sync_In} renamed P1_ADC_~{Sync_In}
- net P2_ADC_~{Sync_Out} renamed P1_ADC_~{Sync_Out}
- net P2_POLL_MOSI renamed P2_AUX_MOSI
- net P2_POLL_SCLK renamed P2_AUX_SCLK
- new net: R?.1, R?.2, U15.7 (WP)
- new net: R?.1, U?.2 (DIR)
- new net AD7794_DOUT: U14.23 (DOUT/~{RDY}), U?.20 (B2)
- new net AD7794_FCLK: U14.2 (CLK), U?.21 (B1)
- new net AD7794_~{CS}: U14.3 (~{CS}), U?.19 (B3)
- new net P1_3P3VAUX: C?.1, R?.1, R?.1, R?.1, U15.8 (VCC)
- new net P1_GA0: U15.1 (A0), U15.2 (A1)
- new net P1_SCL: R?.2, U15.6 (SCL)
- new net P1_SDA: R?.2, U15.5 (SDA)
- new net P2_AD7794_DOUT: U?.4 (A2)
- new net P2_AD7794_FCLK: U?.3 (A1)
- new net P2_AD7794_~{CS}: U?.5 (A3)
- new net Temp_Bridge1/GND: R?.2, U14.14 (REFIN1-)
- new net Temp_Bridge1/VIN: R?.1, U14.13 (REFIN1+)
- new net Temp_Bridge1/Vout+: U14.7 (AIN1+)
- new net Temp_Bridge1/Vout-: U14.8 (AIN1-)
- new net Temp_Bridge2/Vout+: U14.9 (AIN2+)
- new net Temp_Bridge2/Vout-: U14.10 (AIN2-)
- new net Temp_Bridge3/Vout+: U14.11 (AIN3+)
- new net Temp_Bridge3/Vout-: U14.12 (AIN3-)
- new net Temp_Bridge4/Vout+: U14.17 (AIN4+/REFIN2+)
- new net Temp_Bridge4/Vout-: U14.18 (AIN4-/REFIN2-)
- new net VSS3P3V: C?.1, R?.2, U14.21 (AVDD), U14.22 (DVDD)
Other:
- added sheet Temp_Bridge1 (Temp_Bridge.kicad_sch)
- added sheet Temp_Bridge2 (Temp_Bridge.kicad_sch)
- added sheet Temp_Bridge3 (Temp_Bridge.kicad_sch)
- added sheet Temp_Bridge4 (Temp_Bridge.kicad_sch)
- moved on the sheet: C?, U123

Commit message: Updated Schematics with recent changes
Made Updates with recent suggestions.
Parts:
- removed C? (x8): 100nF, symbol Device:C_Small
- removed R? (x2): 4.75k, symbol Device:R_Small_US
- removed U? (x4): 74LVC8T245, symbol Custom_Lib_MPEX_Zest:74LVC8T245
- added C28 (x2): 100nF, symbol Device:C_Small
- added R18 (x2), R? (x2): 4.75k, symbol Device:R_Small_US
- added R?: 22k, symbol Device:R_Small_US
- added U19: 74AVC4T245, symbol Custom_Lib_MPEX_Zest:74LVC4T245
Connections:
- net +5V is gone; now on net VDD3P3V: C?.1, C?.1, C?.1, C?.1, C?.1, C?.1, C?.1, C?.1, U123.1 (~{RESET}), U123.1 (~{RESET}), U123.1 (~{RESET}), U123.1 (~{RESET}), U123.1 (~{RESET}), U123.1 (~{RESET}), U123.1 (~{RESET}), U123.1 (~{RESET})
- net AD7768_~{Sync_In} is gone; now on net ADC1_DCLK: U?.20 (B2)
- net MAX4896_~{FLAG}1 is gone; now on net Relay_SetCoil3: U123.15 (~{FLAG})
- net MAX4896_~{FLAG}2 is gone; now on net Relay_ResetCoil3: U123.15 (~{FLAG})
- net MAX4896_~{FLAG}3 is gone; now on net Relay_SetCoil11: U123.15 (~{FLAG})
- net MAX4896_~{FLAG}4 is gone; now on net Relay_ResetCoil11: U123.15 (~{FLAG})
- net MAX4896_~{FLAG}5 is gone; now on net Relay_SetCoil19: U123.15 (~{FLAG})
- net MAX4896_~{FLAG}6 is gone; now on net Relay_ResetCoil19: U123.15 (~{FLAG})
- net MAX4896_~{FLAG}7 is gone; now on net Relay_SetCoil27: U123.15 (~{FLAG})
- net MAX4896_~{FLAG}8 is gone; now on net Relay_ResetCoil27: U123.15 (~{FLAG})
- net P1_ADC_~{Sync_In} is gone; now on net P1_ADC1_DCLK: U?.4 (A2)
- net AD3: now also R?.1, R?.2
- net AD7768_SCLK: now also U?.16 (B6)
- net AD7768_~{RESET}: now also U?.15 (B7)
- net AD7794_DOUT: now also U19.12 (B2)
- net AD7794_FCLK: now also U19.10 (B4)
- net AD7794_~{CS}: now also U19.11 (B3)
- net ADC1_DCLK: no longer U?.19 (B3)
- net ADC2_DCLK: now also U?.19 (B3); no longer U?.18 (B4)
- net ADC3_DCLK: now also U?.18 (B4); no longer U?.17 (B5)
- net ADC4_DCLK: now also U?.17 (B5); no longer U?.16 (B6)
- net AMC7823_SPI_MISO: now also U19.13 (B1); no longer U?.18 (B4)
- net GND: now also C28.1, C28.1, R18.2, R?.2, R?.2, U19.14 (OE), U19.15 (OE), U19.8 (GND), U19.9 (GND); no longer U?.2 (DIR)
- net P1_ADC1_DCLK: no longer U?.5 (A3)
- net P1_ADC2_DCLK: now also U?.5 (A3); no longer U?.6 (A4)
- net P1_ADC_SCLK: now also U?.8 (A6)
- net P1_ADC_~{RESET}: now also U?.9 (A7)
- net P2_AD7794_DOUT: now also U19.5 (A2)
- net P2_AD7794_FCLK: now also U19.7 (A4)
- net P2_AD7794_~{CS}: now also U19.6 (A3)
- net P2_ADC3_DCLK: now also U?.6 (A4); no longer U?.7 (A5)
- net P2_ADC4_DCLK: now also U?.7 (A5); no longer U?.8 (A6)
- net P2_AMC7823_SPI_MISO: now also U19.4 (A1); no longer U?.6 (A4)
- net P2_VADJ: now also C28.2, R18.2, U19.1 (VCCA)
- net VDD3P3V: now also C28.2, U19.16 (VCCB)
- net AD1 renamed V2P2V_Mon
- net AD2 renamed V3P7V_Mon
- net AMC7823_SPI_MOSI renamed AD7794_DIN
- net AMC7823_SPI_SCLK renamed AD7794_SCLK
- new net: R18.1, U19.3 (2DIR)
- new net: R18.1, U19.2 (1DIR)
- new net: R?.1, U?.2 (DIR)
- new net V12P0V_bus: R?.1
- no-connect marks 0 -> 12
Other:
- moved on the sheet: C?, R?, U14, U15, U?

Commit message: Schmatic Updates
Updated:
ADC MCLK signal
Removed PMOD connectors
Added Coax input for iRIG signal with 5V buffer
Moved around FMC pin mapping
Changed relay driver chip daisy chain order
Changed all input AFE to new design based around the INA851 chip
Parts:
- added C28 (x6): 100nF, symbol Device:C_Small
- added J8: IRIG IN, symbol Connector:Conn_Coaxial
- added R18 (x4): 4.75k, symbol Device:R_Small_US
- added U19 (x2): 74AVC4T245, symbol Custom_Lib_MPEX_Zest:74LVC4T245
- added U38: SN74LVC1T45DBV, Package_TO_SOT_SMD:SOT-23-6, symbol Logic_LevelTranslator:SN74LVC1T45DBV
Connections:
- net GND: now also C28.1, C28.1, C28.1, C28.1, C28.1, C28.1, J8.2 (Ext), R18.2, R18.2, U19.14 (OE), U19.14 (OE), U19.15 (OE), U19.15 (OE), U19.8 (GND), U19.8 (GND), U19.9 (GND), U19.9 (GND), U38.2 (GND), U38.5 (DIR)
- net P2_VADJ: now also C28.2, C28.2, C28.2, R18.2, R18.2, U19.1 (VCCA), U19.1 (VCCA), U38.1 (VCCA)
- net Relay_ResetCoil1: now also U123.18 (OUT1); no longer U123.18 (OUT1)
- net Relay_ResetCoil10: now also U123.17 (OUT2); no longer U123.17 (OUT2)
- net Relay_ResetCoil11: now also U123.15 (~{FLAG}); no longer U123.15 (~{FLAG})
- net Relay_ResetCoil12: now also U123.14 (OUT4); no longer U123.14 (OUT4)
- net Relay_ResetCoil13: now also U123.12 (OUT5); no longer U123.12 (OUT5)
- net Relay_ResetCoil14: now also U123.11 (OUT6); no longer U123.11 (OUT6)
- net Relay_ResetCoil15: now also U123.9 (OUT7); no longer U123.9 (OUT7)
- net Relay_ResetCoil16: now also U123.8 (OUT8); no longer U123.8 (OUT8)
- net Relay_ResetCoil17: now also U123.18 (OUT1); no longer U123.18 (OUT1)
- net Relay_ResetCoil18: now also U123.17 (OUT2); no longer U123.17 (OUT2)
- net Relay_ResetCoil19: now also U123.15 (~{FLAG}); no longer U123.15 (~{FLAG})
- net Relay_ResetCoil2: now also U123.17 (OUT2); no longer U123.17 (OUT2)
- net Relay_ResetCoil20: now also U123.14 (OUT4); no longer U123.14 (OUT4)
- net Relay_ResetCoil21: now also U123.12 (OUT5); no longer U123.12 (OUT5)
- net Relay_ResetCoil22: now also U123.11 (OUT6); no longer U123.11 (OUT6)
- net Relay_ResetCoil23: now also U123.9 (OUT7); no longer U123.9 (OUT7)
- net Relay_ResetCoil24: now also U123.8 (OUT8); no longer U123.8 (OUT8)
- net Relay_ResetCoil3: now also U123.15 (~{FLAG}); no longer U123.15 (~{FLAG})
- net Relay_ResetCoil4: now also U123.14 (OUT4); no longer U123.14 (OUT4)
- net Relay_ResetCoil5: now also U123.12 (OUT5); no longer U123.12 (OUT5)
- net Relay_ResetCoil6: now also U123.11 (OUT6); no longer U123.11 (OUT6)
- net Relay_ResetCoil7: now also U123.9 (OUT7); no longer U123.9 (OUT7)
- net Relay_ResetCoil8: now also U123.8 (OUT8); no longer U123.8 (OUT8)
- net Relay_ResetCoil9: now also U123.18 (OUT1); no longer U123.18 (OUT1)
- net Relay_SetCoil10: now also U123.17 (OUT2); no longer U123.17 (OUT2)
- net Relay_SetCoil11: now also U123.15 (~{FLAG}); no longer U123.15 (~{FLAG})
- net Relay_SetCoil12: now also U123.14 (OUT4); no longer U123.14 (OUT4)
- net Relay_SetCoil13: now also U123.12 (OUT5); no longer U123.12 (OUT5)
- net Relay_SetCoil14: now also U123.11 (OUT6); no longer U123.11 (OUT6)
- net Relay_SetCoil15: now also U123.9 (OUT7); no longer U123.9 (OUT7)
- net Relay_SetCoil16: now also U123.8 (OUT8); no longer U123.8 (OUT8)
- net Relay_SetCoil17: now also U123.18 (OUT1); no longer U123.18 (OUT1)
- net Relay_SetCoil18: now also U123.17 (OUT2); no longer U123.17 (OUT2)
- net Relay_SetCoil19: now also U123.15 (~{FLAG}); no longer U123.15 (~{FLAG})
- net Relay_SetCoil20: now also U123.14 (OUT4); no longer U123.14 (OUT4)
- net Relay_SetCoil21: now also U123.12 (OUT5); no longer U123.12 (OUT5)
- net Relay_SetCoil22: now also U123.11 (OUT6); no longer U123.11 (OUT6)
- net Relay_SetCoil23: now also U123.9 (OUT7); no longer U123.9 (OUT7)
- net Relay_SetCoil24: now also U123.8 (OUT8); no longer U123.8 (OUT8)
- net Relay_SetCoil25: now also U123.18 (OUT1); no longer U123.18 (OUT1)
- net Relay_SetCoil26: now also U123.17 (OUT2); no longer U123.17 (OUT2)
- net Relay_SetCoil27: now also U123.15 (~{FLAG}); no longer U123.15 (~{FLAG})
- net Relay_SetCoil28: now also U123.14 (OUT4); no longer U123.14 (OUT4)
- net Relay_SetCoil29: now also U123.12 (OUT5); no longer U123.12 (OUT5)
- net Relay_SetCoil30: now also U123.11 (OUT6); no longer U123.11 (OUT6)
- net Relay_SetCoil31: now also U123.9 (OUT7); no longer U123.9 (OUT7)
- net Relay_SetCoil32: now also U123.8 (OUT8); no longer U123.8 (OUT8)
- net Relay_SetCoil9: now also U123.18 (OUT1); no longer U123.18 (OUT1)
- net VDD1P8V: now also C28.2, U19.16 (VCCB)
- net VDD3P3V: now also C28.2, C28.2, U19.16 (VCCB), U38.6 (VCCB)
- net Relay_ShiftData_DOUT: now reaches U123.5 (DOUT)
- net Relay_ShiftData_DOUT: now also U19.13 (B1)
- new net: R18.1, U19.2 (1DIR) (x2)
- new net: J8.1 (In), U38.4 (B)
- new net: R18.1, U19.3 (2DIR) (x2)
- new net AD7768_MCLK+: U19.13 (B1)
- new net AD7768_MCLK-: U19.12 (B2)
- new net P2_AD7768_MCLK+: U19.4 (A1)
- new net P2_AD7768_MCLK-: U19.5 (A2)
- new net P2_Relay_ShiftData_DOUT: U19.4 (A1)
- new net P2_Timing_Input: U38.3 (A)
- no-connect marks 12 -> 22
Other:
- moved on the sheet: C?, R?, U15

Commit message: Updated Schematics
Changes:
-Moved Input resistors to after Coupling Relay
-Added diff cap at ADC input
-Changed the ADC clocking configuration (added quad LVDS driver)
-Changed some signal names for consistancy
Parts:
- removed C28 (x4): 100nF, symbol Device:C_Small
- removed C?: 1uF, Capacitor_SMD:C_0603_1608Metric, symbol Device:C_Small
- removed R18 (x4): 4.75k, symbol Device:R_Small_US
- removed R? (x2): 0R, symbol Device:R_Small_US
- removed U14: AD7794, Package_SO:TSSOP-24_4.4x7.8mm_P0.65mm, symbol Analog_ADC:AD7794
- removed U19 (x2): 74AVC4T245, symbol Custom_Lib_MPEX_Zest:74LVC4T245
- added C28: 100nF, symbol Device:C_Small
- added R18 (x2): 4.75k, symbol Device:R_Small_US
- added U20: DSLVDS1047, Package_SO:TSSOP-16_4.4x5mm_P0.65mm, symbol Interface:SN65LVDS047PW
Connections:
- net AD7794_DOUT is gone; now on net Relay_ShiftData_DOUT: U19.12 (B2)
- net P2_AD7794_DOUT is gone; now on net P2_Relay_ShiftData_DOUT: U19.5 (A2)
- net GND: now also C28.1, R18.2, U20.5 (GND)
- net VDD3P3V: now also C28.2, R18.2, U20.4 (VCC)
- net AD7794_DIN renamed AMC7823_SPI_MOSI
- net AD7794_FCLK: no longer names the net of U19.10 (B4)
- net AD7794_SCLK renamed AMC7823_SPI_SCLK
- net AD7794_~{CS}: no longer names the net of U19.11 (B3)
- net ADC1_SDI renamed AD7768_SDI
- net ADC2_SDI: no longer names the net of U?.16 (B6)
- net ADC3_SDI: no longer names the net of U?.15 (B7)
- net ADC4_SDI: no longer names the net of U?.14 (B8)
- removed net MAX4896_Reset: U123.1 (~{RESET}), U123.1 (~{RESET}), U123.1 (~{RESET}), U123.1 (~{RESET}), U123.1 (~{RESET}), U123.1 (~{RESET}), U123.1 (~{RESET}), U123.1 (~{RESET}), U?.17 (B5)
- net P1_ADC1_SDI renamed P1_AD7768_SDI
- net P1_ADC2_SDI: no longer names the net of U?.8 (A6)
- net P2_AD7794_FCLK: no longer names the net of U19.7 (A4)
- net P2_AD7794_~{CS}: no longer names the net of U19.6 (A3)
- net P2_ADC3_SDI: no longer names the net of U?.9 (A7)
- net P2_ADC4_SDI: no longer names the net of U?.10 (A8)
- net P2_MAX4896_Reset renamed P2_MAX4896_~{Reset}
- new net: R18.1, U20.1 (EN)
- new net: R18.1, U20.8 (~{EN})
- new net ADC1_MCLK+: U20.15 (DOUT1+)
- new net ADC1_MCLK-: U20.16 (DOUT1-)
- new net ADC2_MCLK+: U20.14 (DOUT2+)
- new net ADC2_MCLK-: U20.13 (DOUT2-)
- new net ADC3_MCLK+: U20.11 (DOUT3+)
- new net ADC3_MCLK-: U20.12 (DOUT3-)
- new net ADC4_MCLK+: U20.10 (DOUT4+)
- new net ADC4_MCLK-: U20.9 (DOUT4-)
- new net MAX4896_~{Reset}: U123.1 (~{RESET}), U123.1 (~{RESET}), U123.1 (~{RESET}), U123.1 (~{RESET}), U123.1 (~{RESET}), U123.1 (~{RESET}), U123.1 (~{RESET}), U123.1 (~{RESET}), U?.17 (B5)
- new net P2_AD7768_MCLK_LVCMOS: U20.2 (DIN1), U20.3 (DIN2), U20.6 (DIN3), U20.7 (DIN4)
- no-connect marks 22 -> 12
Other:
- removed sheet Temp_Bridge1
- removed sheet Temp_Bridge2
- removed sheet Temp_Bridge3
- removed sheet Temp_Bridge4

Commit message: Updated Schematics with latest suggestions
updates:
-Revised Power supply section
-Changed clock buffer chip for ADC Clock
- Added additional no pop & jumper parts for board debugging
-Other small part changes
Parts:
- removed C28: 100nF, symbol Device:C_Small
- removed C?: 150pF, symbol Device:C_Small
- removed U20: DSLVDS1047, Package_SO:TSSOP-16_4.4x5mm_P0.65mm, symbol Interface:SN65LVDS047PW
- added C? (x2): 100nF, symbol Device:C_Small
- added U3701: SI5330B-B00206-GM, symbol AD7768_Digitizer_SLib:Si5330x
- R18: value 4.75k -> 1k
Connections:
- net AD0: now also C?.1, J?.7 (Pin_7); no longer J?.9 (Pin_9)
- net AD3: now also C?.1, J?.1 (Pin_1); no longer C?.1, J?.3 (Pin_3), R?.1, R?.2
- net AD5: now also R?.1, R?.2
- net ADC1_MCLK+: now also U3701.22 (CLK0A)
- net ADC1_MCLK-: now also U3701.21 (CLK0B)
- net ADC2_MCLK+: now also U3701.18 (CLK1A)
- net ADC2_MCLK-: now also U3701.17 (CLK1B)
- net ADC3_MCLK+: now also U3701.10 (CLK3A)
- net ADC3_MCLK-: now also U3701.9 (CLK3B)
- net ADC4_MCLK+: now also U3701.14 (CLK2A)
- net ADC4_MCLK-: now also U3701.13 (CLK2B)
- net DAC4: now also J?.9 (Pin_9)
- net GND: now also C?.1, C?.1, U3701.12 (GND), U3701.23 (GND), U3701.3 (In3), U3701.4 (GND), U3701.5 (GND), U3701.6 (GND)
- net P2_VADJ: now also R18.2, C?.2, C?.2, U3701.24 (VDD), U3701.7 (VDD)
- net VDD1P8V: now also U3701.11 (VDDO3), U3701.15 (VDDO2), U3701.16 (VDDO1), U3701.20 (VDDO0)
- net VDD3P3V: no longer R18.2
- net P1_ValidCLK: now reaches R18.1
- net P1_ValidCLK: now also U3701.8 (LOS)
- net at R18.1: now also U3701.19 (OEB)
- removed net AD4: C?.1, J?.1 (Pin_1), U?.17 (CH4)
- removed net V2P2V_Mon: C?.1, J?.7 (Pin_7), U?.12 (CH1)
- net V3P7V_Mon renamed AD1
- net AD1: now also U?.12 (CH1); no longer U?.13 (CH2)
- new net 2P3V_Mon: U?.17 (CH4)
- new net AD2: C?.1, J?.3 (Pin_3), U?.13 (CH2)
- new net P1_AD7768_MCLK+: U3701.1 (In1)
- new net P1_AD7768_MCLK-: U3701.2 (In2)
Other:
- moved on the sheet: C28, C?, J8, R18, R?, U15, U38
