File: Housekeeping.kicad_sch (KiCad schematic)
At the start: 96 parts, among them J5 PPS IN, J6 WP Jumper, Q1 FDN335N, Q2 FDN335N, U123 MAX4896, U15 AT24C64D-SSHM, U16 SI5330B-B00206-GM, U19 74AVC4T245, U36 TL071H, U37 TXU0101

Commit message: Update to Schematics; initial PCB commit
-Updated Power, Housekeeping, and ADCs sheets.
-Remapped FMC pins
-Initial board layout commit
Parts:
- removed U123 (x7): MAX4896, symbol AD7768_Digitizer_SLib:MAX4896
- added C? (x4): 100nF, Capacitor_SMD:C_0402_1005Metric, symbol Device:C_Small
- added U123 (x7): MAX4896, Package_DFN_QFN:TQFN-20-1EP_5x5mm_P0.65mm_EP3.1x3.1mm, symbol AD7768_Digitizer_SLib:MAX4896
- C? (x6): footprint Capacitor_SMD:C_0603_1608Metric -> Capacitor_SMD:C_0402_1005Metric
- C? (x3): footprint (none) -> Capacitor_SMD:C_0402_1005Metric
- D3: footprint (none) -> LED_SMD:LED_0603_1608Metric; MPN (none) -> APT1608CGCK
- D?: MPN LTST-C190GKT -> APT1608CGCK
- J6: footprint (none) -> Connector_PinSocket_2.00mm:PinSocket_1x02_P2.00mm_Vertical
- J? (x2): footprint (none) -> Connector_PinHeader_1.27mm:PinHeader_2x10_P1.27mm_Vertical_SMD
- Q1, Q2: footprint (none) -> Package_TO_SOT_SMD:SOT-23
- R18, R? (x10): footprint (none) -> Resistor_SMD:R_0402_1005Metric
- R18: value 1k -> 100R; footprint (none) -> Resistor_SMD:R_0402_1005Metric
- R? (x5): footprint Resistor_SMD:R_0603_1608Metric -> Resistor_SMD:R_0402_1005Metric
- R?: footprint (none) -> Resistor_SMD:R_0603_1608Metric
- U123: footprint (none) -> Package_DFN_QFN:TQFN-20-1EP_5x5mm_P0.65mm_EP3.1x3.1mm
- U16: footprint (none) -> Package_DFN_QFN:QFN-24-1EP_4x4mm_P0.5mm_EP2.6x2.6mm
- U19: footprint (none) -> Package_SO:TSSOP-16_4.4x5mm_P0.65mm
- U36: footprint (none) -> Package_TO_SOT_SMD:SOT-23-5
- U? (x4): footprint (none) -> Package_SO:TSSOP-24_4.4x7.8mm_P0.65mm
- U?: footprint QFN50P600X600X80-41N -> Package_DFN_QFN:QFN-40-1EP_6x6mm_P0.5mm_EP4.6x4.6mm
Connections:
- net PGND is gone; now on net GND: U123.16 (PGND)
- net 15V+: now also C?.2
- net 15V-: now also C?.2
- net ADC1_MCLK+: now also U16.10 (CLK3A); no longer U16.22 (CLK0A)
- net ADC1_MCLK-: now also U16.9 (CLK3B); no longer U16.21 (CLK0B)
- net ADC2_MCLK+: now also U16.14 (CLK2A); no longer U16.18 (CLK1A)
- net ADC2_MCLK-: now also U16.13 (CLK2B); no longer U16.17 (CLK1B)
- net ADC3_MCLK+: now also U16.18 (CLK1A); no longer U16.10 (CLK3A)
- net ADC3_MCLK-: now also U16.17 (CLK1B); no longer U16.9 (CLK3B)
- net ADC4_MCLK+: now also U16.22 (CLK0A); no longer U16.14 (CLK2A)
- net ADC4_MCLK-: now also U16.21 (CLK0B); no longer U16.13 (CLK2B)
- net GND: now also U16.19 (OEB), U19.6 (A3), U19.7 (A4), U?.6 (A4), C?.1, C?.1, U123.10 (PGND), U123.10 (PGND), U123.10 (PGND), U123.10 (PGND), U123.10 (PGND), U123.10 (PGND), U123.10 (PGND), U123.13 (GND), U123.13 (GND), U123.13 (GND), U123.13 (GND), U123.13 (GND), U123.13 (GND), U123.13 (GND), U123.16 (PGND), U123.16 (PGND), U123.16 (PGND), U123.16 (PGND), U123.16 (PGND), U123.16 (PGND), U123.16 (PGND), U123.21 (EP), U123.21 (EP), U123.21 (EP), U123.21 (EP), U123.21 (EP), U123.21 (EP), U123.21 (EP), U123.6 (PDCD), U123.6 (PDCD), U123.6 (PDCD), U123.6 (PDCD), U123.6 (PDCD), U123.6 (PDCD), U123.6 (PDCD), U123.7 (SPLD), U123.7 (SPLD), U123.7 (SPLD), U123.7 (SPLD), U123.7 (SPLD), U123.7 (SPLD), U123.7 (SPLD); no longer R18.2
- net MAX4896_SCLK: now also U123.4 (SCLK), U123.4 (SCLK), U123.4 (SCLK), U123.4 (SCLK), U123.4 (SCLK), U123.4 (SCLK), U123.4 (SCLK)
- net MAX4896_~{CS}: now also U123.2 (~{CS}), U123.2 (~{CS}), U123.2 (~{CS}), U123.2 (~{CS}), U123.2 (~{CS}), U123.2 (~{CS}), U123.2 (~{CS})
- net MAX4896_~{Reset}: now also U123.1 (~{RESET}), U123.1 (~{RESET}), U123.1 (~{RESET}), U123.1 (~{RESET}), U123.1 (~{RESET}), U123.1 (~{RESET}), U123.1 (~{RESET})
- net Relay_ResetCoil1: now also U123.18 (OUT1)
- net Relay_ResetCoil10: now also U123.17 (OUT2)
- net Relay_ResetCoil11: now also U123.15 (OUT3)
- net Relay_ResetCoil12: now also U123.14 (OUT4)
- net Relay_ResetCoil13: now also U123.12 (OUT5)
- net Relay_ResetCoil14: now also U123.11 (OUT6)
- net Relay_ResetCoil15: now also U123.9 (OUT7)
- net Relay_ResetCoil16: now also U123.8 (OUT8)
- net Relay_ResetCoil17: now also U123.18 (OUT1)
- net Relay_ResetCoil18: now also U123.17 (OUT2)
- net Relay_ResetCoil19: now also U123.15 (OUT3)
- net Relay_ResetCoil2: now also U123.17 (OUT2)
- net Relay_ResetCoil20: now also U123.14 (OUT4)
- net Relay_ResetCoil21: now also U123.12 (OUT5)
- net Relay_ResetCoil22: now also U123.11 (OUT6)
- net Relay_ResetCoil23: now also U123.9 (OUT7)
- net Relay_ResetCoil24: now also U123.8 (OUT8)
- net Relay_ResetCoil25: now also U123.18 (OUT1)
- net Relay_ResetCoil26: now also U123.17 (OUT2)
- net Relay_ResetCoil27: now also U123.15 (OUT3)
- net Relay_ResetCoil28: now also U123.14 (OUT4)
- net Relay_ResetCoil29: now also U123.12 (OUT5)
- net Relay_ResetCoil3: now also U123.15 (OUT3)
- net Relay_ResetCoil30: now also U123.11 (OUT6)
- net Relay_ResetCoil31: now also U123.9 (OUT7)
- net Relay_ResetCoil32: now also U123.8 (OUT8)
- net Relay_ResetCoil4: now also U123.14 (OUT4)
- net Relay_ResetCoil5: now also U123.12 (OUT5)
- net Relay_ResetCoil6: now also U123.11 (OUT6)
- net Relay_ResetCoil7: now also U123.9 (OUT7)
- net Relay_ResetCoil8: now also U123.8 (OUT8)
- net Relay_ResetCoil9: now also U123.18 (OUT1)
- net Relay_SetCoil10: now also U123.17 (OUT2)
- net Relay_SetCoil11: now also U123.15 (OUT3)
- net Relay_SetCoil12: now also U123.14 (OUT4)
- net Relay_SetCoil13: now also U123.12 (OUT5)
- net Relay_SetCoil14: now also U123.11 (OUT6)
- net Relay_SetCoil15: now also U123.9 (OUT7)
- net Relay_SetCoil16: now also U123.8 (OUT8)
- net Relay_SetCoil17: now also U123.18 (OUT1)
- net Relay_SetCoil18: now also U123.17 (OUT2)
- net Relay_SetCoil19: now also U123.15 (OUT3)
- net Relay_SetCoil20: now also U123.14 (OUT4)
- net Relay_SetCoil21: now also U123.12 (OUT5)
- net Relay_SetCoil22: now also U123.11 (OUT6)
- net Relay_SetCoil23: now also U123.9 (OUT7)
- net Relay_SetCoil24: now also U123.8 (OUT8)
- net Relay_SetCoil25: now also U123.18 (OUT1)
- net Relay_SetCoil26: now also U123.17 (OUT2)
- net Relay_SetCoil27: now also U123.15 (OUT3)
- net Relay_SetCoil28: now also U123.14 (OUT4)
- net Relay_SetCoil29: now also U123.12 (OUT5)
- net Relay_SetCoil30: now also U123.11 (OUT6)
- net Relay_SetCoil31: now also U123.9 (OUT7)
- net Relay_SetCoil32: now also U123.8 (OUT8)
- net Relay_SetCoil9: now also U123.18 (OUT1)
- net Relay_ShiftData_DOUT: now also U123.5 (DOUT)
- net VDD3P3V: now also U123.19 (Vs), U123.19 (Vs), U123.19 (Vs), U123.19 (Vs), U123.19 (Vs), U123.19 (Vs), U123.19 (Vs), U123.19 (Vs); no longer U123.1 (~{RESET})
- net at U123.5 (DOUT): now also U123.3 (DIN)
- net P2_AD7768_MCLK-: now reaches R18.1
- net P2_AD7768_MCLK-: now also C?.2; no longer U16.19 (OEB)
- net P1_AD7768_MCLK+: no longer names the net of U16.1 (In1)
- net P1_AD7768_MCLK+: now also C?.1
- net P1_AD7768_MCLK-: no longer names the net of U16.2 (In2)
- net P1_AD7768_MCLK-: now also C?.1
- net P1_ValidCLK renamed P2_ValidCLK
- new net: U123.3 (DIN), U123.5 (DOUT) (x6)
- new net P2_AD7768_MCLK+: C?.2, R18.2
- no-connect marks 12 -> 13
Other:
- moved on the sheet: R?

Commit message: Updated Layout
-Additional Layout Work
Parts:
- removed R18 (x2), R?: 4.75k, Resistor_SMD:R_0402_1005Metric, symbol Device:R_Small_US
- added C? (x4): 100nF, Capacitor_SMD:C_0402_1005Metric, symbol Device:C_Small
- added R18: 10k, Resistor_SMD:R_0402_1005Metric, symbol Device:R_Small_US
- C28, C? (x2): footprint (none) -> Capacitor_SMD:C_0402_1005Metric
- C? (x6): footprint Capacitor_SMD:C_0603_1608Metric -> Capacitor_SMD:C_0402_1005Metric
- J5: footprint (none) -> Connector_Coaxial:SMA_Amphenol_901-144_Vertical
Connections:
- net AD7768_SCLK: now also U?.15 (B7); no longer U?.16 (B6)
- net AD7768_SDI: now also U?.16 (B6); no longer U?.17 (B5)
- net AD7768_~{RESET}: now also U?.18 (B4); no longer U?.15 (B7)
- net AD7768_~{Start}: now also U?.19 (B3); no longer U?.21 (B1)
- net ADC1_DCLK: now also U?.17 (B5); no longer U?.20 (B2)
- net ADC1_SDO: now also U?.14 (B8); no longer U?.17 (B5)
- net ADC1_~{CS}: now also U?.14 (B8); no longer U?.21 (B1)
- net ADC1_~{DRDY}: now also U?.15 (B7); no longer U?.21 (B1)
- net ADC2_DCLK: now also U?.21 (B1); no longer U?.19 (B3)
- net ADC2_~{CS}: now also U?.20 (B2); no longer U?.20 (B2)
- net ADC2_~{DRDY}: now also U?.17 (B5); no longer U?.20 (B2)
- net ADC3_DCLK: now also U?.15 (B7); no longer U?.18 (B4)
- net ADC3_SDO: now also U?.18 (B4); no longer U?.15 (B7)
- net ADC3_~{CS}: now also U?.14 (B8); no longer U?.19 (B3)
- net ADC4_DCLK: now also U?.19 (B3); no longer U?.17 (B5)
- net ADC4_SDO: now also U?.20 (B2); no longer U?.14 (B8)
- net ADC4_~{DRDY}: now also U?.21 (B1); no longer U?.18 (B4)
- net GND: now also U16.25 (GND), U19.10 (B4), U19.2 (1DIR), U19.3 (2DIR), U?.2 (DIR), C?.1, C?.1, C?.1, C?.1; no longer U19.6 (A3)
- net P1_AD7768_SDI: now also U?.8 (A6); no longer U?.7 (A5)
- net P1_ADC1_DCLK: now also U?.7 (A5); no longer U?.4 (A2)
- net P1_ADC1_SDO: now also U?.10 (A8); no longer U?.7 (A5)
- net P1_ADC1_~{CS}: now also U?.10 (A8); no longer U?.3 (A1)
- net P1_ADC1_~{DRDY}: now also U?.9 (A7); no longer U?.3 (A1)
- net P1_ADC2_DCLK: now also U?.3 (A1); no longer U?.5 (A3)
- net P1_ADC2_~{CS}: now also U?.4 (A2); no longer U?.4 (A2)
- net P1_ADC2_~{DRDY}: now also U?.7 (A5); no longer U?.4 (A2)
- net P1_ADC_SCLK: now also U?.9 (A7); no longer U?.8 (A6)
- net P1_ADC_~{RESET}: now also U?.6 (A4); no longer U?.9 (A7)
- net P1_ADC_~{Start}: now also U?.5 (A3); no longer U?.3 (A1)
- net P2_ADC3_DCLK: now also U?.9 (A7); no longer U?.6 (A4)
- net P2_ADC3_SDO: now also U?.6 (A4); no longer U?.9 (A7)
- net P2_ADC3_~{CS}: now also U?.10 (A8); no longer U?.5 (A3)
- net P2_ADC4_DCLK: no longer U?.7 (A5)
- net P2_ADC4_SDO: now also U?.4 (A2); no longer U?.10 (A8)
- net P2_ADC4_~{DRDY}: now also U?.3 (A1); no longer U?.6 (A4)
- net VDD1P8V: now also C?.2, C?.2, C?.2, C?.2
- net VDD3P3V: now also R18.1
- net MAX4896_~{Flag}: now reaches U19.11 (B3)
- net MAX4896_~{Flag}: now also U123.20 (~{FLAG}), U123.20 (~{FLAG}), U123.20 (~{FLAG}), U123.20 (~{FLAG}), U123.20 (~{FLAG}), U123.20 (~{FLAG}), U123.20 (~{FLAG}), U123.20 (~{FLAG}), R18.2
- new net P2_MAX4896_~{Flag}: U19.6 (A3)
- no-connect marks 13 -> 1

Commit message: Updated Schematics with all suggestions
-Added pull up resistors on SDO line to FPGA
-Fixed some I/O flags to properly indicate direction
-Added Bulk caps on 15V rails
-Added series caps to AC couple the LVDS clock lines. See AN408 from the manufacture
-Add Voltage monitor for 1.8V and 5V
Parts:
- removed C? (x5): 150pF, Capacitor_SMD:C_0402_1005Metric, symbol Device:C_Small
- added C? (x4): 100nF, Capacitor_SMD:C_0402_1005Metric, symbol Device:C_Small
- added H1, H2: MountingHole, MountingHole:MountingHole_3mm, symbol Mechanical:MountingHole
- added R? (x5): 10k, Resistor_SMD:R_0402_1005Metric, symbol Device:R_Small_US
- added R? (x2): 4.75k, Resistor_SMD:R_0603_1608Metric, symbol Device:R_Small_US
- added R?: 390R, Resistor_SMD:R_0603_1608Metric, symbol Device:R_Small_US
- added R?: 10k, Resistor_SMD:R_0603_1608Metric, symbol Device:R_Small_US
- R? (x2): value 200R -> 1k
Connections:
- net +5V: now also R?.1
- net AD0: now also C?.2, J?.1 (Pin_1); no longer J?.3 (Pin_3)
- net AD1: now also R?.1, R?.2; no longer C?.2, J?.1 (Pin_1)
- net ADC1_SDO: now also R?.2
- net ADC2_SDO: now also R?.2
- net ADC3_SDO: now also R?.2
- net ADC4_SDO: now also R?.2
- net AMC7823_SPI_MISO: now also R?.2
- net DAC7: now also J?.3 (Pin_3)
- net GND: now also C?.1, C?.1, C?.1, C?.1, R?.2, R?.2
- net VDD1P8V: now also R?.1, R?.1, R?.1, R?.1, R?.1
- net VDD3P3V: now also C?.2, C?.2, C?.2, C?.2, R?.1
- net 2P3V_Mon renamed AD4
- net AD4: now also R?.1, R?.2
Other:
- moved on the sheet: C28, C?, R?, U19, U?

Commit message: Updated Project
Schematics:
-updated level shifting IC's
-Add notes to level shifters
-Changed Relay Coil Driver channel mapping
-Added additional Mounting Hole

Layout
-WIP To Complete:
-Relay Driver ICs
- Reworking LT8582 area
- Level Shifters
- Housekeeping ICs
-Misc. error cleanup
- Silkscreen adjust
- Add Silkscreen SN & logo
Parts:
- removed C? (x2): 100nF, Capacitor_SMD:C_0402_1005Metric, symbol Device:C_Small
- removed R? (x2): 10k, Resistor_SMD:R_0402_1005Metric, symbol Device:R_Small_US
- removed U? (x2): 74LVC8T245, Package_SO:TSSOP-24_4.4x7.8mm_P0.65mm, symbol Custom_Lib_MPEX_Zest:74LVC8T245
- added C? (x4): 100nF, Capacitor_SMD:C_0402_1005Metric, symbol Device:C_Small
- added H2: MountingHole, MountingHole:MountingHole_3mm, symbol Mechanical:MountingHole
- added R? (x2): 10k, Resistor_SMD:R_0402_1005Metric, symbol Device:R_Small_US
- added R?: 4.75k, Resistor_SMD:R_0402_1005Metric, symbol Device:R_Small_US
- added U19 (x3): 74AVC4T245, Package_SO:TSSOP-16_4.4x5mm_P0.65mm, symbol Custom_Lib_MPEX_Zest:74LVC4T245
Connections:
- net ADC1_SDO: now also R?.2, U19.10 (B4)
- net ADC1_~{DRDY}: now also U19.11 (B3)
- net ADC2_SDO: now also R?.2, U19.12 (B2)
- net ADC2_~{DRDY}: now also U19.13 (B1)
- net ADC3_DCLK: now also U19.11 (B3)
- net ADC3_SDO: now also U19.10 (B4)
- net ADC3_~{CS}: now also U19.10 (B4)
- net ADC3_~{DRDY}: now also U19.11 (B3)
- net ADC4_DCLK: now also U19.13 (B1)
- net ADC4_SDO: now also U19.12 (B2)
- net ADC4_~{CS}: now also U19.12 (B2)
- net ADC4_~{DRDY}: now also U19.13 (B1)
- net GND: now also C?.2, C?.2, C?.2, C?.2, U19.14 (OE), U19.14 (OE), U19.14 (OE), U19.15 (OE), U19.15 (OE), U19.15 (OE), U19.2 (1DIR), U19.2 (1DIR), U19.3 (2DIR), U19.3 (2DIR), U19.8 (GND), U19.8 (GND), U19.8 (GND), U19.9 (GND), U19.9 (GND), U19.9 (GND)
- net P1_ADC1_SDO: now also U19.7 (A4)
- net P1_ADC1_~{DRDY}: now also U19.6 (A3)
- net P1_ADC2_SDO: now also U19.5 (A2)
- net P1_ADC2_~{DRDY}: now also U19.4 (A1)
- net P2_ADC3_DCLK: now also U19.6 (A3)
- net P2_ADC3_SDO: now also U19.7 (A4)
- net P2_ADC3_~{CS}: now also U19.7 (A4)
- net P2_ADC3_~{DRDY}: now also U19.6 (A3)
- net P2_ADC4_DCLK: now also U19.4 (A1)
- net P2_ADC4_SDO: now also U19.5 (A2)
- net P2_ADC4_~{CS}: now also U19.5 (A2)
- net P2_ADC4_~{DRDY}: now also U19.4 (A1)
- net P2_VADJ: now also C?.1, R?.2, U19.1 (VCCA), U19.1 (VCCA); no longer C?.1, R?.2, U?.1 (VCCA)
- net Relay_ResetCoil1: now also U123.15 (OUT3); no longer U123.18 (OUT1)
- net Relay_ResetCoil10: now also U123.9 (OUT7); no longer U123.17 (OUT2)
- net Relay_ResetCoil11: now also U123.15 (OUT3); no longer U123.15 (OUT3)
- net Relay_ResetCoil12: now also U123.9 (OUT7); no longer U123.14 (OUT4)
- net Relay_ResetCoil13: now also U123.18 (OUT1); no longer U123.12 (OUT5)
- net Relay_ResetCoil14: now also U123.12 (OUT5); no longer U123.11 (OUT6)
- net Relay_ResetCoil15: now also U123.18 (OUT1); no longer U123.9 (OUT7)
- net Relay_ResetCoil16: now also U123.12 (OUT5); no longer U123.8 (OUT8)
- net Relay_ResetCoil17: now also U123.15 (OUT3); no longer U123.18 (OUT1)
- net Relay_ResetCoil18: now also U123.9 (OUT7); no longer U123.17 (OUT2)
- net Relay_ResetCoil19: now also U123.15 (OUT3); no longer U123.15 (OUT3)
- net Relay_ResetCoil2: now also U123.9 (OUT7); no longer U123.17 (OUT2)
- net Relay_ResetCoil20: now also U123.9 (OUT7); no longer U123.14 (OUT4)
- net Relay_ResetCoil21: now also U123.18 (OUT1); no longer U123.12 (OUT5)
- net Relay_ResetCoil22: now also U123.12 (OUT5); no longer U123.11 (OUT6)
- net Relay_ResetCoil23: now also U123.18 (OUT1); no longer U123.9 (OUT7)
- net Relay_ResetCoil24: now also U123.12 (OUT5); no longer U123.8 (OUT8)
- net Relay_ResetCoil25: now also U123.15 (OUT3); no longer U123.18 (OUT1)
- net Relay_ResetCoil26: now also U123.9 (OUT7); no longer U123.17 (OUT2)
- net Relay_ResetCoil28: now also U123.9 (OUT7); no longer U123.14 (OUT4)
- net Relay_ResetCoil29: now also U123.18 (OUT1); no longer U123.12 (OUT5)
- net Relay_ResetCoil3: now also U123.15 (OUT3); no longer U123.15 (OUT3)
- net Relay_ResetCoil30: now also U123.12 (OUT5); no longer U123.11 (OUT6)
- net Relay_ResetCoil31: now also U123.18 (OUT1); no longer U123.9 (OUT7)
- net Relay_ResetCoil32: now also U123.12 (OUT5); no longer U123.8 (OUT8)
- net Relay_ResetCoil4: now also U123.9 (OUT7); no longer U123.14 (OUT4)
- net Relay_ResetCoil5: now also U123.18 (OUT1); no longer U123.12 (OUT5)
- net Relay_ResetCoil6: now also U123.12 (OUT5); no longer U123.11 (OUT6)
- net Relay_ResetCoil7: now also U123.18 (OUT1); no longer U123.9 (OUT7)
- net Relay_ResetCoil8: now also U123.12 (OUT5); no longer U123.8 (OUT8)
- net Relay_ResetCoil9: now also U123.15 (OUT3); no longer U123.18 (OUT1)
- net Relay_SetCoil1: now also U123.14 (OUT4); no longer U123.18 (OUT1)
- net Relay_SetCoil10: now also U123.8 (OUT8); no longer U123.17 (OUT2)
- net Relay_SetCoil11: now also U123.14 (OUT4); no longer U123.15 (OUT3)
- net Relay_SetCoil12: now also U123.8 (OUT8); no longer U123.14 (OUT4)
- net Relay_SetCoil13: now also U123.17 (OUT2); no longer U123.12 (OUT5)
- net Relay_SetCoil14: now also U123.11 (OUT6); no longer U123.11 (OUT6)
- net Relay_SetCoil15: now also U123.17 (OUT2); no longer U123.9 (OUT7)
- net Relay_SetCoil16: now also U123.11 (OUT6); no longer U123.8 (OUT8)
- net Relay_SetCoil17: now also U123.14 (OUT4); no longer U123.18 (OUT1)
- net Relay_SetCoil18: now also U123.8 (OUT8); no longer U123.17 (OUT2)
- net Relay_SetCoil19: now also U123.14 (OUT4); no longer U123.15 (OUT3)
- net Relay_SetCoil2: now also U123.8 (OUT8); no longer U123.17 (OUT2)
- net Relay_SetCoil20: now also U123.8 (OUT8); no longer U123.14 (OUT4)
- net Relay_SetCoil21: now also U123.17 (OUT2); no longer U123.12 (OUT5)
- net Relay_SetCoil22: now also U123.11 (OUT6); no longer U123.11 (OUT6)
- net Relay_SetCoil23: now also U123.17 (OUT2); no longer U123.9 (OUT7)
- net Relay_SetCoil24: now also U123.11 (OUT6); no longer U123.8 (OUT8)
- net Relay_SetCoil25: now also U123.14 (OUT4); no longer U123.18 (OUT1)
- net Relay_SetCoil26: now also U123.8 (OUT8); no longer U123.17 (OUT2)
- net Relay_SetCoil27: now also U123.14 (OUT4); no longer U123.15 (OUT3)
- net Relay_SetCoil28: now also U123.8 (OUT8); no longer U123.14 (OUT4)
- net Relay_SetCoil29: now also U123.17 (OUT2); no longer U123.12 (OUT5)
- net Relay_SetCoil3: now also U123.14 (OUT4); no longer U123.15 (OUT3)
- net Relay_SetCoil30: now also U123.11 (OUT6); no longer U123.11 (OUT6)
- net Relay_SetCoil31: now also U123.17 (OUT2); no longer U123.9 (OUT7)
- net Relay_SetCoil32: now also U123.11 (OUT6); no longer U123.8 (OUT8)
- net Relay_SetCoil4: now also U123.8 (OUT8); no longer U123.14 (OUT4)
- net Relay_SetCoil5: now also U123.17 (OUT2); no longer U123.12 (OUT5)
- net Relay_SetCoil7: now also U123.17 (OUT2); no longer U123.9 (OUT7)
- net Relay_SetCoil8: now also U123.11 (OUT6); no longer U123.8 (OUT8)
- net Relay_SetCoil9: now also U123.14 (OUT4); no longer U123.18 (OUT1)
- net VDD1P8V: now also C?.1, C?.1, R?.1, R?.1, U19.16 (VCCB), U19.16 (VCCB), U19.16 (VCCB)
- net at R?.1: now also U19.2 (1DIR)
- new net: R?.1, U19.3 (2DIR)
- new net P1_VADJ: C?.1, C?.1, R?.2, U19.1 (VCCA), U?.1 (VCCA)
Other:
- note added: "+2.5V"
- note added: "From ADCs"
- note added: "From FPGA"
- note added: "From On-Board IC's"
- note added: "PPS Timing Input"
- note added: "To ADCs"
- note added: "To FPGA"
- note added: "To On-Board IC's"
- moved on the sheet: C28, C?, H1, H2, J5, R?, U19, U37, U?

Commit message: Updated Project with Latest Changes
Project:
-Added pdf plots of PCB layout

Schematics:
-Fixed L8 Pinout
-Adjusted FMC connections
-Adjusted level shifter connections

Layout:
-Completed AFE/ADC/Power/Relay driver sections

Layout WIP To Complete:
-Misc. error cleanup
- Silkscreen adjust
- Add Silkscreen SN & logo
Connections:
- net AMC7823_SPI_MOSI: now also U?.20 (B2); no longer U?.19 (B3)
- net AMC7823_SPI_SCLK: now also U?.21 (B1); no longer U?.20 (B2)
- net AMC7823_SPI_SS: now also U?.19 (B3); no longer U?.21 (B1)
- net GND: now also U123.11 (OUT6), U123.9 (OUT7); no longer U123.13 (GND), U123.6 (PDCD), U123.7 (SPLD)
- net MAX4896_SCLK: now also U?.17 (B5); no longer U123.4 (SCLK), U?.16 (B6)
- net MAX4896_~{CS}: now also U?.16 (B6); no longer U123.2 (~{CS}), U?.15 (B7)
- net MAX4896_~{Flag}: now also U19.12 (B2); no longer U123.20 (~{FLAG}), U19.11 (B3)
- net MAX4896_~{Reset}: now also U?.15 (B7); no longer U123.1 (~{RESET}), U?.17 (B5)
- net P2_AMC7823_SPI_MOSI: now also U?.4 (A2); no longer U?.5 (A3)
- net P2_AMC7823_SPI_SCLK: now also U?.3 (A1); no longer U?.4 (A2)
- net P2_AMC7823_SPI_SS: now also U?.5 (A3); no longer U?.3 (A1)
- net P2_MAX4896_SCLK: now also U?.7 (A5); no longer U?.8 (A6)
- net P2_MAX4896_~{CS}: now also U?.8 (A6); no longer U?.9 (A7)
- net P2_MAX4896_~{Flag}: now also U19.5 (A2); no longer U19.6 (A3)
- net P2_MAX4896_~{Reset}: now also U?.9 (A7); no longer U?.7 (A5)
- net P2_Relay_ShiftData_DOUT: now also U19.6 (A3); no longer U19.5 (A2)
- net Relay_ResetCoil3: no longer U123.15 (OUT3)
- net Relay_ResetCoil4: no longer U123.9 (OUT7)
- net Relay_ResetCoil7: no longer U123.18 (OUT1)
- net Relay_ResetCoil8: no longer U123.12 (OUT5)
- net Relay_SetCoil3: no longer U123.14 (OUT4)
- net Relay_SetCoil4: no longer U123.8 (OUT8)
- net Relay_SetCoil7: no longer U123.17 (OUT2)
- net Relay_SetCoil8: no longer U123.11 (OUT6)
- net Relay_ShiftData_DOUT: now also U19.11 (B3); no longer U19.12 (B2)
- net at U123.5 (DOUT): now also U123.5 (DOUT); no longer U123.3 (DIN)
- net at U123.3 (DIN): no longer U123.5 (DOUT)
Other:
- moved on the sheet: U123
