File: Quartz_v1p1.kicad_pcb (KiCad board)
At the start: 6 copper layers, 254 x 130 mm, 1249 parts, among them J1 5747847-6, J2 5747847-6, J3 Conn_02x10_Odd_Even, J4 Conn_02x10_Odd_Even, J5 PPS IN, J6 WP Jumper, K1001 EE2-12TNU-L, K101 EE2-12TNU-L, K1101 EE2-12TNU-L, K1201 EE2-12TNU-L, K1301 EE2-12TNU-L, K1401 EE2-12TNU-L, K1501 EE2-12TNU-L, K1601 EE2-12TNU-L, K1701 EE2-12TNU-L, K1801 EE2-12TNU-L, K1901 EE2-12TNU-L, K2001 EE2-12TNU-L, K201 EE2-12TNU-L, K2101 EE2-12TNU-L, K2201 EE2-12TNU-L, K2301 EE2-12TNU-L, K2401 EE2-12TNU-L, K2501 EE2-12TNU-L, K2601 EE2-12TNU-L, K2701 EE2-12TNU-L, K2801 EE2-12TNU-L, K2901 EE2-12TNU-L, K3001 EE2-12TNU-L, K301 EE2-12TNU-L, K3101 EE2-12TNU-L, K3201 EE2-12TNU-L, K401 EE2-12TNU-L, K501 EE2-12TNU-L, K601 EE2-12TNU-L, K701 EE2-12TNU-L, K801 EE2-12TNU-L, K901 EE2-12TNU-L, P1 ASP-134604-01, P2 ASP-134604-01, Q1 FDN335N, Q2 FDN335N, Q3 FDMC510P, U1 AD7768, U10 AD7768, U1001 INA851, U101 INA851, U11 ADR4540, U1101 INA851, U12 ADA4841-1, U1201 INA851, U13 AMC7823IRTAR, U1301 INA851, U14 MAX4896, U1401 INA851, U15 MAX4896, U1501 INA851, U16 SI5330B-B00206-GM, U1601 INA851, U17 MAX4896, U1701 INA851, U18 MAX4896, U1801 INA851, U19 MAX4896, U1901 INA851, U2 ADR4540, U20 MAX4896, U2001 INA851, U201 INA851, U21 MAX4896, U2101 INA851, U22 74AVC4T245, U2201 INA851, U23 MAX4896, U2301 INA851, U24 74AVC4T245, U2401 INA851, U25 74LVC8T245, U2501 INA851, U26 74AVC4T245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

Commit message: Updated Project with Latest Changes
Project:
-Added pdf plots of PCB layout

Schematics:
-Fixed L8 Pinout
-Adjusted FMC connections
-Adjusted level shifter connections

Layout:
-Completed AFE/ADC/Power/Relay driver sections

Layout WIP To Complete:
-Misc. error cleanup
- Silkscreen adjust
- Add Silkscreen SN & logo
Parts:
- removed C174, C175, C176, C177: 10uF, Capacitor_SMD:C_0805_2012Metric
- C156, C161, C162, C166, C170, R111, R81, R89, R92, U34: moved to F.Cu
- C157: moved to B.Cu
- R1, R2, R3: footprint Resistor_SMD:R_0603_1608Metric -> Resistor_SMD:R_0402_1005Metric
- U1001, U101, U1101, U1201, U1301, U1401, U1501, U1601, U1701, U1801, U1901, U2001, U201, U2101, U2201, U2301, U2401, U2501, U2601, U2701, U2801, U2901, U3001, U301, U3101, U3201, U401, U501, U601, U701, U801, U901: footprint Package_DFN_QFN:QFN-16-1EP_3x3mm_P0.5mm_EP1.75x1.75mm_ThermalVias -> footprints:QFN-16-1EP_3x3mm_P0.5mm_EP1.75x1.75mm_ThermalVias
- moved C126 88.7 mm to (186.9, 163.2), turned to 90 degrees
- moved C95 76.3 mm to (225.9, 163.2), turned to 90 degrees
- moved C152 73.8 mm to (214.6, 112.9)
- moved L5 73.8 mm to (211.7, 112.0)
- moved TP10 73.8 mm to (217.7, 116.0)
- moved TP4 73.8 mm to (217.7, 111.9)
- moved D6 73.8 mm to (212.2, 116.2)
- moved R76 73.8 mm to (208.3, 111.9)
- moved R78 73.8 mm to (210.7, 114.6)
- moved C117 66.3 mm to (252.2, 163.2), turned to 90 degrees
- moved C121 66.0 mm to (164.2, 163.2), turned to 90 degrees
- moved C122 40.3 mm to (276.7, 163.2), turned to 90 degrees
- moved C116 36.1 mm to (137.9, 163.2), turned to 90 degrees
- moved C127 32.1 mm to (313.4, 163.2), turned to 90 degrees
- moved C154 27.7 mm to (102.6, 143.0)
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Connections:
- net /ADC1/ADC_VCM renamed /ADC_VCM1
- net /ADC2/ADC_VCM renamed /ADC_VCM2
- net /ADC3/ADC_VCM renamed /ADC_VCM3
- net /ADC4/ADC_VCM renamed /ADC_VCM4
- net /Channel01/Housekeeping_INA_Out+ renamed /Channel01/FMC_INA_Out+
- net /Channel01/Housekeeping_INA_Out- renamed /Channel01/FMC_INA_Out-
- net /Channel02/Housekeeping_INA_Out+ renamed /Channel02/FMC_INA_Out+
- net /Channel02/Housekeeping_INA_Out- renamed /Channel02/FMC_INA_Out-
- net /Channel03/Housekeeping_INA_Out+ renamed /Channel03/FMC_INA_Out+
- net /Channel03/Housekeeping_INA_Out- renamed /Channel03/FMC_INA_Out-
- net /Channel04/Housekeeping_INA_Out+ renamed /Channel04/FMC_INA_Out+
- net /Channel04/Housekeeping_INA_Out- renamed /Channel04/FMC_INA_Out-
- net /Channel05/Housekeeping_INA_Out+ renamed /Channel05/FMC_INA_Out+
- net /Channel05/Housekeeping_INA_Out- renamed /Channel05/FMC_INA_Out-
- net /Channel06/Housekeeping_INA_Out+ renamed /Channel06/FMC_INA_Out+
- net /Channel06/Housekeeping_INA_Out- renamed /Channel06/FMC_INA_Out-
- net /Channel07/Housekeeping_INA_Out+ renamed /Channel07/FMC_INA_Out+
- net /Channel07/Housekeeping_INA_Out- renamed /Channel07/FMC_INA_Out-
- net /Channel08/Housekeeping_INA_Out+ renamed /Channel08/FMC_INA_Out+
- net /Channel08/Housekeeping_INA_Out- renamed /Channel08/FMC_INA_Out-
- net /Channel09/Housekeeping_INA_Out+ renamed /Channel09/FMC_INA_Out+
- net /Channel09/Housekeeping_INA_Out- renamed /Channel09/FMC_INA_Out-
- net /Channel10/Housekeeping_INA_Out+ renamed /Channel10/FMC_INA_Out+
- net /Channel10/Housekeeping_INA_Out- renamed /Channel10/FMC_INA_Out-
- net /Channel11/Housekeeping_INA_Out+ renamed /Channel11/FMC_INA_Out+
- net /Channel11/Housekeeping_INA_Out- renamed /Channel11/FMC_INA_Out-
- net /Channel12/Housekeeping_INA_Out+ renamed /Channel12/FMC_INA_Out+
- net /Channel12/Housekeeping_INA_Out- renamed /Channel12/FMC_INA_Out-
- net /Channel13/Housekeeping_INA_Out+ renamed /Channel13/FMC_INA_Out+
- net /Channel13/Housekeeping_INA_Out- renamed /Channel13/FMC_INA_Out-
- net /Channel14/Housekeeping_INA_Out+ renamed /Channel14/FMC_INA_Out+
- net /Channel14/Housekeeping_INA_Out- renamed /Channel14/FMC_INA_Out-
- net /Channel15/Housekeeping_INA_Out+ renamed /Channel15/FMC_INA_Out+
- net /Channel15/Housekeeping_INA_Out- renamed /Channel15/FMC_INA_Out-
- net /Channel16/Housekeeping_INA_Out+ renamed /Channel16/FMC_INA_Out+
- net /Channel16/Housekeeping_INA_Out- renamed /Channel16/FMC_INA_Out-
- net /Channel17/Housekeeping_INA_Out+ renamed /Channel17/FMC_INA_Out+
- net /Channel17/Housekeeping_INA_Out- renamed /Channel17/FMC_INA_Out-
- net /Channel18/Housekeeping_INA_Out+ renamed /Channel18/FMC_INA_Out+
- net /Channel18/Housekeeping_INA_Out- renamed /Channel18/FMC_INA_Out-
- net /Channel19/Housekeeping_INA_Out+ renamed /Channel19/FMC_INA_Out+
- net /Channel19/Housekeeping_INA_Out- renamed /Channel19/FMC_INA_Out-
- net /Channel20/Housekeeping_INA_Out+ renamed /Channel20/FMC_INA_Out+
- net /Channel20/Housekeeping_INA_Out- renamed /Channel20/FMC_INA_Out-
- net /Channel21/Housekeeping_INA_Out+ renamed /Channel21/FMC_INA_Out+
- net /Channel21/Housekeeping_INA_Out- renamed /Channel21/FMC_INA_Out-
- net /Channel22/Housekeeping_INA_Out+ renamed /Channel22/FMC_INA_Out+
- net /Channel22/Housekeeping_INA_Out- renamed /Channel22/FMC_INA_Out-
- net /Channel23/Housekeeping_INA_Out+ renamed /Channel23/FMC_INA_Out+
- net /Channel23/Housekeeping_INA_Out- renamed /Channel23/FMC_INA_Out-
- net /Channel24/Housekeeping_INA_Out+ renamed /Channel24/FMC_INA_Out+
- net /Channel24/Housekeeping_INA_Out- renamed /Channel24/FMC_INA_Out-
- net /Channel25/Housekeeping_INA_Out+ renamed /Channel25/FMC_INA_Out+
- net /Channel25/Housekeeping_INA_Out- renamed /Channel25/FMC_INA_Out-
- net /Channel26/Housekeeping_INA_Out+ renamed /Channel26/FMC_INA_Out+
- net /Channel26/Housekeeping_INA_Out- renamed /Channel26/FMC_INA_Out-
- net /Channel27/Housekeeping_INA_Out+ renamed /Channel27/FMC_INA_Out+
- net /Channel27/Housekeeping_INA_Out- renamed /Channel27/FMC_INA_Out-
- net /Channel28/Housekeeping_INA_Out+ renamed /Channel28/FMC_INA_Out+
- net /Channel28/Housekeeping_INA_Out- renamed /Channel28/FMC_INA_Out-
- net /Channel29/Housekeeping_INA_Out+ renamed /Channel29/FMC_INA_Out+
- net /Channel29/Housekeeping_INA_Out- renamed /Channel29/FMC_INA_Out-
- net /Channel30/Housekeeping_INA_Out+ renamed /Channel30/FMC_INA_Out+
- net /Channel30/Housekeeping_INA_Out- renamed /Channel30/FMC_INA_Out-
- net /Channel31/Housekeeping_INA_Out+ renamed /Channel31/FMC_INA_Out+
- net /Channel31/Housekeeping_INA_Out- renamed /Channel31/FMC_INA_Out-
- net /Channel32/Housekeeping_INA_Out+ renamed /Channel32/FMC_INA_Out+
- net /Channel32/Housekeeping_INA_Out- renamed /Channel32/FMC_INA_Out-
- L8 pad 2: Net-(U35-SWA2) -> Net-(L8-Pad2)
- L8 pad 3: Net-(L8-Pad3) -> Net-(U35-SWA2)
- P1 pad D20: P2_MAX4896_~{Reset} -> unconnected-(P1-PadD20)
- P1 pad D21: P2_MAX4896_SCLK -> unconnected-(P1-PadD21)
- P1 pad D23: P2_Relay_ShiftData_DOUT -> unconnected-(P1-PadD23)
- P1 pad D24: P2_Relay_ShiftData -> unconnected-(P1-PadD24)
- P1 pad D26: P2_MAX4896_~{CS} -> unconnected-(P1-PadD26)
- P2 pad D8: P2_MAX4896_~{Flag} -> P2_Timing_Input
- P2 pad D9: unconnected-(P2-PadD9) -> P2_ValidCLK
- P2 pad G10: P2_AMC7823_SPI_MOSI -> P2_AMC7823_SPI_SCLK
- P2 pad G12: P2_AMC7823_SPI_MISO -> P2_AMC7823_SPI_MOSI
- P2 pad G15: unconnected-(P2-PadG15) -> P2_MAX4896_SCLK
- P2 pad G16: unconnected-(P2-PadG16) -> P2_MAX4896_~{CS}
- P2 pad G18: unconnected-(P2-PadG18) -> P2_MAX4896_~{Reset}
- P2 pad G19: unconnected-(P2-PadG19) -> P2_Relay_ShiftData
- P2 pad G6: P2_Timing_Input -> P2_AMC7823_SPI_MISO
- P2 pad G7: P2_ValidCLK -> P2_MAX4896_~{Flag}
- P2 pad G9: P2_AMC7823_SPI_SCLK -> P2_Relay_ShiftData_DOUT
- R110 pad 2: Net-(L8-Pad3) -> Net-(L8-Pad2)
- R99 pad 1: Net-(L8-Pad3) -> Net-(L8-Pad2)
- U17 pad 1: MAX4896_~{Reset} -> unconnected-(U17-~{RESET}-Pad1)
- U17 pad 11: /Relay_SetCoil8 -> GND
- U17 pad 12: /Relay_ResetCoil8 -> unconnected-(U17-OUT5-Pad12)
- U17 pad 13: GND -> unconnected-(U17-GND-Pad13)
- U17 pad 14: /Relay_SetCoil3 -> unconnected-(U17-OUT4-Pad14)
- U17 pad 15: /Relay_ResetCoil3 -> unconnected-(U17-OUT3-Pad15)
- U17 pad 17: /Relay_SetCoil7 -> unconnected-(U17-OUT2-Pad17)
- U17 pad 18: /Relay_ResetCoil7 -> unconnected-(U17-OUT1-Pad18)
- U17 pad 2: MAX4896_~{CS} -> unconnected-(U17-~{CS}-Pad2)
- U17 pad 20: MAX4896_~{Flag} -> unconnected-(U17-~{FLAG}-Pad20)
- U17 pad 3: Net-(U14-DOUT) -> unconnected-(U17-DIN-Pad3)
- U17 pad 4: MAX4896_SCLK -> unconnected-(U17-SCLK-Pad4)
- U17 pad 5: Net-(U17-DOUT) -> Net-(U14-DOUT)
- U17 pad 6: GND -> unconnected-(U17-PDCD-Pad6)
- U17 pad 7: GND -> unconnected-(U17-SPLD-Pad7)
- U17 pad 8: /Relay_SetCoil4 -> unconnected-(U17-OUT8-Pad8)
- U17 pad 9: /Relay_ResetCoil4 -> GND
- U19 pad 3: Net-(U17-DOUT) -> unconnected-(U19-DIN-Pad3)
- U26 pad 11: MAX4896_~{Flag} -> Relay_ShiftData_DOUT
- U26 pad 12: Relay_ShiftData_DOUT -> MAX4896_~{Flag}
- U26 pad 5: P2_Relay_ShiftData_DOUT -> P2_MAX4896_~{Flag}
- U26 pad 6: P2_MAX4896_~{Flag} -> P2_Relay_ShiftData_DOUT
- U29 pad 15: MAX4896_~{CS} -> MAX4896_~{Reset}
- U29 pad 16: MAX4896_SCLK -> MAX4896_~{CS}
- U29 pad 17: MAX4896_~{Reset} -> MAX4896_SCLK
- U29 pad 19: AMC7823_SPI_MOSI -> AMC7823_SPI_SS
- U29 pad 20: AMC7823_SPI_SCLK -> AMC7823_SPI_MOSI
- U29 pad 21: AMC7823_SPI_SS -> AMC7823_SPI_SCLK
- U29 pad 3: P2_AMC7823_SPI_SS -> P2_AMC7823_SPI_SCLK
- U29 pad 4: P2_AMC7823_SPI_SCLK -> P2_AMC7823_SPI_MOSI
- U29 pad 5: P2_AMC7823_SPI_MOSI -> P2_AMC7823_SPI_SS
- U29 pad 7: P2_MAX4896_~{Reset} -> P2_MAX4896_SCLK
- U29 pad 8: P2_MAX4896_SCLK -> P2_MAX4896_~{CS}
- U29 pad 9: P2_MAX4896_~{CS} -> P2_MAX4896_~{Reset}
Routing:
- net +5V: track 356.9 -> 767.9 mm, vias 67 -> 83
- net VDD3P3V: track 0.00 -> 362.7 mm, vias 0 -> 8
- net MAX4896_~{Reset}: track 0.00 -> 269.0 mm, vias 0 -> 8
- net MAX4896_~{CS}: track 0.00 -> 265.7 mm, vias 0 -> 9
- net MAX4896_SCLK: track 0.00 -> 261.7 mm, vias 0 -> 9
- net MAX4896_~{Flag}: track 0.00 -> 260.0 mm, vias 0 -> 8
- net GND: track 671.0 -> 904.0 mm, vias 399 -> 484
- net Relay_ShiftData: track 0.00 -> 217.4 mm, vias 0 -> 2
- net /ADC_SYNC: track 4.11 -> 149.3 mm, vias 0 -> 4
- net /ADC_VCM3: track 18.7 -> 143.6 mm, vias 0 -> 9
- net /ADC_VCM1: track 18.7 -> 131.9 mm, vias 0 -> 11
- net /ADC_VCM2: track 18.7 -> 128.1 mm, vias 0 -> 9
- net /ADC_VCM4: track 18.7 -> 117.4 mm, vias 0 -> 9
- net AD7768_~{RESET}: track 39.3 -> 130.2 mm, vias 1 -> 4
- net Relay_ShiftData_DOUT: track 0.00 -> 56.6 mm, vias 0 -> 1
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- added copper zone on In2.Cu, net +12V
- added copper zone on F.Cu, net /Power/-16V
- added copper zone on F.Cu, net /Power/16V
- added copper zone on In2.Cu, net /Power/LT8582_VIN
- added copper zone on In2.Cu, net 15V+
- added copper zone on In2.Cu, net 15V-
- removed copper zone on B.Cu, net /Power/16V
