File: Quartz_v1p1.kicad_pcb (KiCad board)
At the start: 6 copper layers, 254 x 130 mm, 1245 parts, among them J1 5747847-6, J2 5747847-6, J3 Conn_02x10_Odd_Even, J4 Conn_02x10_Odd_Even, J5 PPS IN, J6 WP Jumper, K1001 EE2-12TNU-L, K101 EE2-12TNU-L, K1101 EE2-12TNU-L, K1201 EE2-12TNU-L, K1301 EE2-12TNU-L, K1401 EE2-12TNU-L, K1501 EE2-12TNU-L, K1601 EE2-12TNU-L, K1701 EE2-12TNU-L, K1801 EE2-12TNU-L, K1901 EE2-12TNU-L, K2001 EE2-12TNU-L, K201 EE2-12TNU-L, K2101 EE2-12TNU-L, K2201 EE2-12TNU-L, K2301 EE2-12TNU-L, K2401 EE2-12TNU-L, K2501 EE2-12TNU-L, K2601 EE2-12TNU-L, K2701 EE2-12TNU-L, K2801 EE2-12TNU-L, K2901 EE2-12TNU-L, K3001 EE2-12TNU-L, K301 EE2-12TNU-L, K3101 EE2-12TNU-L, K3201 EE2-12TNU-L, K401 EE2-12TNU-L, K501 EE2-12TNU-L, K601 EE2-12TNU-L, K701 EE2-12TNU-L, K801 EE2-12TNU-L, K901 EE2-12TNU-L, P1 ASP-134604-01, P2 ASP-134604-01, Q1 FDN335N, Q2 FDN335N, Q3 FDMC510P, U1 AD7768, U10 AD7768, U1001 INA851, U101 INA851, U11 ADR4540, U1101 INA851, U12 ADA4841-1, U1201 INA851, U13 AMC7823IRTAR, U1301 INA851, U14 MAX4896, U1401 INA851, U15 MAX4896, U1501 INA851, U16 SI5330B-B00206-GM, U1601 INA851, U17 MAX4896, U1701 INA851, U18 MAX4896, U1801 INA851, U19 MAX4896, U1901 INA851, U2 ADR4540, U20 MAX4896, U2001 INA851, U201 INA851, U21 MAX4896, U2101 INA851, U22 74AVC4T245, U2201 INA851, U23 MAX4896, U2301 INA851, U24 74AVC4T245, U2401 INA851, U25 74LVC8T245, U2501 INA851, U26 74AVC4T245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

Commit message: Changed ADCs to run on +2.5V VADJ
Modified schematic to allow the ADCs to be run from the +2.5V VADJ inputs on the FMC connector.
-All relevant ERC issues ran been looked into.
-Still working on all Board DRC issues.
Parts:
- removed C118, C125, C128, C129, C132, C134, C136, C186: 100nF, Capacitor_SMD:C_0402_1005Metric
- removed C139: 10nF, Capacitor_SMD:C_0603_1608Metric
- removed C140, C146, C148: 1uF, Capacitor_SMD:C_0603_1608Metric
- removed C141, C142: 22uF, Capacitor_SMD:C_0805_2012Metric
- removed C143: 10uF, Capacitor_SMD:C_0805_2012Metric
- removed C144: 10pF, Capacitor_SMD:C_0603_1608Metric
- removed C145, C147: 47uF, Capacitor_SMD:C_0805_2012Metric
- removed L1, L3: 120R@100Mhz; 3A, Inductor_SMD:L_0805_2012Metric
- removed L2: 10uH, footprints:IND_7345-WE-PD_WRE
- removed R10: 4.75k, Resistor_SMD:R_0603_1608Metric
- removed R17, R22, R23, R47: 10k, Resistor_SMD:R_0402_1005Metric
- removed R48, R50, R59: 4.75k, Resistor_SMD:R_0402_1005Metric
- removed R5: 390R, Resistor_SMD:R_0603_1608Metric
- removed R63, R64: 0R, Resistor_SMD:R_0603_1608Metric
- removed R66, R68, R70: 422k, Resistor_SMD:R_0603_1608Metric
- removed TP1, TP2: ~, TestPoint:TestPoint_Loop_D1.80mm_Drill1.0mm_Beaded
- removed U22, U24, U28: 74AVC4T245, Package_SO:TSSOP-16_4.4x5mm_P0.65mm
- removed U25: 74LVC8T245, Package_SO:TSSOP-24_4.4x7.8mm_P0.65mm
- removed U30: TPS62110, Package_DFN_QFN:QFN-16-1EP_4x4mm_P0.65mm_EP2.7x2.7mm_PullBack
- removed U31: LT1763, Package_DFN_QFN:DFN-12-1EP_3x4mm_P0.5mm_EP1.7x3.3mm
- moved C169 44.9 mm to (88.2, 124.5), turned to -90 degrees
- moved R79 38.9 mm to (126.5, 118.5), turned to -90 degrees
- moved R98 38.1 mm to (105.9, 117.2), turned to -90 degrees
- moved L8 38.0 mm to (97.4, 121.8), turned to -90 degrees
- moved R93 37.7 mm to (106.9, 117.2), turned to -90 degrees
- moved C163 37.4 mm to (108.0, 117.2), turned to -90 degrees
- moved C159 37.1 mm to (109.0, 117.2), turned to 90 degrees
- moved R91 36.8 mm to (110.0, 117.2), turned to -90 degrees
- moved R83 36.6 mm to (111.0, 117.2), turned to -90 degrees
- moved L6 35.5 mm to (124.9, 120.4), turned to -90 degrees
- moved C153 34.1 mm to (122.9, 120.5), turned to 90 degrees
- moved U35 31.3 mm to (108.7, 121.4), turned to 90 degrees
- moved L7 30.8 mm to (117.3, 121.4), turned to 180 degrees
- moved C164 28.1 mm to (104.0, 125.7), turned to 180 degrees
- moved C168 27.9 mm to (98.8, 130.3), turned to 0 degrees
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Connections:
- net /Channel01/Housekeeping_INA_Out+ renamed /Channel01/Power_INA_Out+
- net /Channel01/Housekeeping_INA_Out- renamed /Channel01/Power_INA_Out-
- net /Channel02/Housekeeping_INA_Out+ renamed /Channel02/Power_INA_Out+
- net /Channel02/Housekeeping_INA_Out- renamed /Channel02/Power_INA_Out-
- net /Channel03/Housekeeping_INA_Out+ renamed /Channel03/Power_INA_Out+
- net /Channel03/Housekeeping_INA_Out- renamed /Channel03/Power_INA_Out-
- net /Channel04/Housekeeping_INA_Out+ renamed /Channel04/Power_INA_Out+
- net /Channel04/Housekeeping_INA_Out- renamed /Channel04/Power_INA_Out-
- net /Channel05/Housekeeping_INA_Out+ renamed /Channel05/Power_INA_Out+
- net /Channel05/Housekeeping_INA_Out- renamed /Channel05/Power_INA_Out-
- net /Channel06/Housekeeping_INA_Out+ renamed /Channel06/Power_INA_Out+
- net /Channel06/Housekeeping_INA_Out- renamed /Channel06/Power_INA_Out-
- net /Channel07/Housekeeping_INA_Out+ renamed /Channel07/Power_INA_Out+
- net /Channel07/Housekeeping_INA_Out- renamed /Channel07/Power_INA_Out-
- net /Channel08/Housekeeping_INA_Out+ renamed /Channel08/Power_INA_Out+
- net /Channel08/Housekeeping_INA_Out- renamed /Channel08/Power_INA_Out-
- net /Channel09/Housekeeping_INA_Out+ renamed /Channel09/Power_INA_Out+
- net /Channel09/Housekeeping_INA_Out- renamed /Channel09/Power_INA_Out-
- net /Channel10/Housekeeping_INA_Out+ renamed /Channel10/Power_INA_Out+
- net /Channel10/Housekeeping_INA_Out- renamed /Channel10/Power_INA_Out-
- net /Channel11/Housekeeping_INA_Out+ renamed /Channel11/Power_INA_Out+
- net /Channel11/Housekeeping_INA_Out- renamed /Channel11/Power_INA_Out-
- net /Channel12/Housekeeping_INA_Out+ renamed /Channel12/Power_INA_Out+
- net /Channel12/Housekeeping_INA_Out- renamed /Channel12/Power_INA_Out-
- net /Channel13/Housekeeping_INA_Out+ renamed /Channel13/Power_INA_Out+
- net /Channel13/Housekeeping_INA_Out- renamed /Channel13/Power_INA_Out-
- net /Channel14/Housekeeping_INA_Out+ renamed /Channel14/Power_INA_Out+
- net /Channel14/Housekeeping_INA_Out- renamed /Channel14/Power_INA_Out-
- net /Channel15/Housekeeping_INA_Out+ renamed /Channel15/Power_INA_Out+
- net /Channel15/Housekeeping_INA_Out- renamed /Channel15/Power_INA_Out-
- net /Channel16/Housekeeping_INA_Out+ renamed /Channel16/Power_INA_Out+
- net /Channel16/Housekeeping_INA_Out- renamed /Channel16/Power_INA_Out-
- net /Channel17/Housekeeping_INA_Out+ renamed /Channel17/Power_INA_Out+
- net /Channel17/Housekeeping_INA_Out- renamed /Channel17/Power_INA_Out-
- net /Channel18/Housekeeping_INA_Out+ renamed /Channel18/Power_INA_Out+
- net /Channel18/Housekeeping_INA_Out- renamed /Channel18/Power_INA_Out-
- net /Channel19/Housekeeping_INA_Out+ renamed /Channel19/Power_INA_Out+
- net /Channel19/Housekeeping_INA_Out- renamed /Channel19/Power_INA_Out-
- net /Channel20/Housekeeping_INA_Out+ renamed /Channel20/Power_INA_Out+
- net /Channel20/Housekeeping_INA_Out- renamed /Channel20/Power_INA_Out-
- net /Channel21/Housekeeping_INA_Out+ renamed /Channel21/Power_INA_Out+
- net /Channel21/Housekeeping_INA_Out- renamed /Channel21/Power_INA_Out-
- net /Channel22/Housekeeping_INA_Out+ renamed /Channel22/Power_INA_Out+
- net /Channel22/Housekeeping_INA_Out- renamed /Channel22/Power_INA_Out-
- net /Channel23/Housekeeping_INA_Out+ renamed /Channel23/Power_INA_Out+
- net /Channel23/Housekeeping_INA_Out- renamed /Channel23/Power_INA_Out-
- net /Channel24/Housekeeping_INA_Out+ renamed /Channel24/Power_INA_Out+
- net /Channel24/Housekeeping_INA_Out- renamed /Channel24/Power_INA_Out-
- net /Channel25/Housekeeping_INA_Out+ renamed /Channel25/Power_INA_Out+
- net /Channel25/Housekeeping_INA_Out- renamed /Channel25/Power_INA_Out-
- net /Channel26/Housekeeping_INA_Out+ renamed /Channel26/Power_INA_Out+
- net /Channel26/Housekeeping_INA_Out- renamed /Channel26/Power_INA_Out-
- net /Channel27/Housekeeping_INA_Out+ renamed /Channel27/Power_INA_Out+
- net /Channel27/Housekeeping_INA_Out- renamed /Channel27/Power_INA_Out-
- net /Channel28/Housekeeping_INA_Out+ renamed /Channel28/Power_INA_Out+
- net /Channel28/Housekeeping_INA_Out- renamed /Channel28/Power_INA_Out-
- net /Channel29/Housekeeping_INA_Out+ renamed /Channel29/Power_INA_Out+
- net /Channel29/Housekeeping_INA_Out- renamed /Channel29/Power_INA_Out-
- net /Channel30/Housekeeping_INA_Out+ renamed /Channel30/Power_INA_Out+
- net /Channel30/Housekeeping_INA_Out- renamed /Channel30/Power_INA_Out-
- net /Channel31/Housekeeping_INA_Out+ renamed /Channel31/Power_INA_Out+
- net /Channel31/Housekeeping_INA_Out- renamed /Channel31/Power_INA_Out-
- net /Channel32/Housekeeping_INA_Out+ renamed /Channel32/Power_INA_Out+
- net /Channel32/Housekeeping_INA_Out- renamed /Channel32/Power_INA_Out-
- C10 pad 1: VDD1P8V -> P1_VADJ
- C11 pad 1: VDD1P8V -> P1_VADJ
- C12 pad 1: VDD1P8V -> P1_VADJ
- C120 pad 2: VDD1P8V -> P2_VADJ
- C171 pad 2: VDD1P8V -> P2_VADJ
- C172 pad 2: VDD1P8V -> P1_VADJ
- C173 pad 2: VDD1P8V -> P1_VADJ
- C29 pad 1: VDD1P8V -> P1_VADJ
- C30 pad 1: VDD1P8V -> P1_VADJ
- C32 pad 1: VDD1P8V -> P1_VADJ
- C33 pad 1: VDD1P8V -> P1_VADJ
- C47 pad 1: VDD1P8V -> P2_VADJ
- C48 pad 1: VDD1P8V -> P2_VADJ
- C51 pad 1: VDD1P8V -> P2_VADJ
- C52 pad 1: VDD1P8V -> P2_VADJ
- C59 pad 1: VDD1P8V -> P2_VADJ
- C60 pad 1: VDD1P8V -> P2_VADJ
- C69 pad 1: VDD1P8V -> P2_VADJ
- C70 pad 1: VDD1P8V -> P2_VADJ
- C9 pad 1: VDD1P8V -> P1_VADJ
- D4 pad 2: I_Mon -> I_MON
- P1 pad G27: P1_ADC2_DCLK -> ADC2_DCLK
- P1 pad G28: P1_ADC2_~{CS} -> ADC2_~{CS}
- P1 pad G30: P1_ADC_~{Start} -> AD7768_~{Start}
- P1 pad G31: P1_ADC_~{RESET} -> AD7768_~{RESET}
- P1 pad G33: P1_ADC1_DCLK -> ADC1_DCLK
- P1 pad G34: P1_AD7768_SDI -> AD7768_SDI
- P1 pad G36: P1_ADC_SCLK -> AD7768_SCLK
- P1 pad G37: P1_ADC1_~{CS} -> ADC1_~{CS}
- P1 pad G6: P1_ADC2_~{DRDY} -> ADC2_~{DRDY}
- P1 pad G7: P1_ADC2_SDO -> ADC2_SDO
- P1 pad H7: P1_ADC1_~{DRDY} -> ADC1_~{DRDY}
- P1 pad H8: P1_ADC1_SDO -> ADC1_SDO
- P2 pad G21: P2_ADC4_~{DRDY} -> ADC4_~{DRDY}
- P2 pad G22: P2_ADC4_SDO -> ADC4_SDO
- P2 pad G24: P2_ADC4_DCLK -> ADC4_DCLK
- P2 pad G25: P2_ADC4_~{CS} -> ADC4_~{CS}
- P2 pad H22: P2_ADC3_~{DRDY} -> ADC3_~{DRDY}
- P2 pad H23: P2_ADC3_SDO -> ADC3_SDO
- P2 pad H25: P2_ADC3_DCLK -> ADC3_DCLK
- P2 pad H26: P2_ADC3_~{CS} -> ADC3_~{CS}
- R1 pad 1: VDD1P8V -> P1_VADJ
- R112 pad 1: VDD1P8V -> P1_VADJ
- R113 pad 1: VDD1P8V -> P1_VADJ
- R114 pad 1: VDD1P8V -> P2_VADJ
- R115 pad 1: VDD1P8V -> P2_VADJ
- R13 pad 1: VDD1P8V -> P1_VADJ
- R19 pad 1: VDD1P8V -> P2_VADJ
- R2 pad 1: VDD1P8V -> P2_VADJ
- R25 pad 1: VDD1P8V -> P2_VADJ
- R3 pad 1: VDD1P8V -> P2_VADJ
- R69 pad 1: I_Mon -> I_MON
- R7 pad 1: VDD1P8V -> P1_VADJ
- U1 pad 34: VDD1P8V -> P1_VADJ
- U1 pad 35: VDD1P8V -> P1_VADJ
- U10 pad 34: VDD1P8V -> P2_VADJ
- U10 pad 35: VDD1P8V -> P2_VADJ
- U16 pad 11: VDD1P8V -> P1_VADJ
- U16 pad 15: VDD1P8V -> P1_VADJ
- U16 pad 16: VDD1P8V -> P2_VADJ
- U16 pad 20: VDD1P8V -> P2_VADJ
- U17 pad 1: unconnected-(U17-~{RESET}-Pad1) -> MAX4896_~{Reset}
- U17 pad 11: GND -> /Relay_SetCoil8
- U17 pad 12: unconnected-(U17-OUT5-Pad12) -> /Relay_ResetCoil8
- U17 pad 13: unconnected-(U17-GND-Pad13) -> GND
- U17 pad 14: unconnected-(U17-OUT4-Pad14) -> /Relay_SetCoil3
- U17 pad 15: unconnected-(U17-OUT3-Pad15) -> /Relay_ResetCoil3
- U17 pad 17: unconnected-(U17-OUT2-Pad17) -> /Relay_SetCoil7
- U17 pad 18: unconnected-(U17-OUT1-Pad18) -> /Relay_ResetCoil7
- U17 pad 2: unconnected-(U17-~{CS}-Pad2) -> MAX4896_~{CS}
- U17 pad 20: unconnected-(U17-~{FLAG}-Pad20) -> MAX4896_~{Flag}
- U17 pad 3: unconnected-(U17-DIN-Pad3) -> Net-(U14-DOUT)
- U17 pad 4: unconnected-(U17-SCLK-Pad4) -> MAX4896_SCLK
- U17 pad 5: Net-(U14-DOUT) -> Net-(U17-DOUT)
- U17 pad 6: unconnected-(U17-PDCD-Pad6) -> GND
- U17 pad 7: unconnected-(U17-SPLD-Pad7) -> GND
- U17 pad 8: unconnected-(U17-OUT8-Pad8) -> /Relay_SetCoil4
- U17 pad 9: GND -> /Relay_ResetCoil4
- U19 pad 3: unconnected-(U19-DIN-Pad3) -> Net-(U17-DOUT)
- U32 pad 1: I_Mon -> I_MON
- U4 pad 34: VDD1P8V -> P1_VADJ
- U4 pad 35: VDD1P8V -> P1_VADJ
- U7 pad 34: VDD1P8V -> P2_VADJ
- U7 pad 35: VDD1P8V -> P2_VADJ
Routing:
- net VDD1P8V: track 389.7 -> 0.00 mm, vias 17 -> 0
- net GND: track 983.2 -> 918.8 mm, vias 526 -> 489
- net +12V: track 967.1 -> 905.1 mm
- net +5V: track 814.2 -> 777.3 mm
- net ADC1_~{CS}: track 44.9 -> 73.1 mm, vias 1 -> 3
- net AD7768_SCLK: track 185.6 -> 213.5 mm, vias 4 -> 6
- net Net-(U14-DOUT): track 42.7 -> 15.4 mm, vias 4 -> 2
- net Net-(U17-DOUT): track 0.00 -> 27.3 mm, vias 0 -> 2
- net AD7768_SDI: track 186.1 -> 213.0 mm, vias 4 -> 6
- net ADC1_DCLK: track 40.3 -> 66.3 mm, vias 1 -> 3
- net /Power/TPS62110_VIN: track 25.1 -> 0.00 mm
- net AD7768_~{RESET}: track 130.2 -> 154.6 mm, vias 4 -> 6
- net AD7768_~{Start}: track 38.7 -> 62.2 mm, vias 1 -> 3
- net P1_ADC1_~{CS}: track 22.2 -> 0.00 mm, vias 2 -> 0
- net P1_ADC_SCLK: track 21.9 -> 0.00 mm, vias 2 -> 0
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- removed copper zone on F.Cu, net /Power/TPS62110_VIN
