File: Quartz_v1p1.kicad_sch (KiCad schematic)
At the start: 5 parts, among them J1 5747847-6, J2 5747847-6

Commit message: Update to Schematics; initial PCB commit
-Updated Power, Housekeeping, and ADCs sheets.
-Remapped FMC pins
-Initial board layout commit
Connections:
- no-connect marks 0 -> 3
Changed lines of the file:
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@@
   (junction (at 361.95 240.03) (diameter 0) (color 0 0 0 0)
   )
+  (no_connect (at 425.45 80.01))
+  (no_connect (at 425.45 232.41))
+  (no_connect (at 232.41 232.41))
   (bus_entry (at 353.06 53.34) (size 2.54 2.54)
     (stroke (width 0) (type default))
@@
     (stroke (width 0) (type default))
   )
-  (wire (pts (xy 199.39 82.55) (xy 182.88 82.55))
-    (stroke (width 0) (type default))
-  )
   (wire (pts (xy 421.64 250.19) (xy 425.45 250.19))
     (stroke (width 0) (type default))
@@
     (stroke (width 0) (type default))
   )
-  (wire (pts (xy 199.39 92.71) (xy 172.72 92.71))
-    (stroke (width 0) (type default))
-  )
   (wire (pts (xy 421.64 123.19) (xy 425.45 123.19))
     (stroke (width 0) (type default))
@@
     (stroke (width 0) (type default))
   )
+  (wire (pts (xy 177.8 87.63) (xy 199.39 87.63))
+    (stroke (width 0) (type default))
+  )
   (wire (pts (xy 228.6 269.24) (xy 232.41 269.24))
     (stroke (width 0) (type default))
@@
     (stroke (width 0) (type default))
   )
-  (wire (pts (xy 199.39 90.17) (xy 175.26 90.17))
-    (stroke (width 0) (type default))
-  )
   (wire (pts (xy 199.39 247.65) (xy 172.72 247.65))
     (stroke (width 0) (type default))
@@
     (stroke (width 0) (type default))
   )
-  (wire (pts (xy 199.39 80.01) (xy 185.42 80.01))
-    (stroke (width 0) (type default))
-  )
   (wire (pts (xy 177.8 273.05) (xy 140.97 273.05))
     (stroke (width 0) (type default))
@@
     (stroke (width 0) (type default))
   )
+  (wire (pts (xy 185.42 80.01) (xy 199.39 80.01))
+    (stroke (width 0) (type default))
+  )
   (bus (pts (xy 162.56 39.37) (xy 162.56 58.42))
     (stroke (width 0) (type default))
@@
     (stroke (width 0) (type default))
   )
+  (wire (pts (xy 172.72 92.71) (xy 199.39 92.71))
+    (stroke (width 0) (type default))
+  )
   (wire (pts (xy 140.97 113.03) (xy 160.02 113.03))
     (stroke (width 0) (type default))
@@
     (stroke (width 0) (type default))
   )
+  (wire (pts (xy 187.96 77.47) (xy 199.39 77.47))
+    (stroke (width 0) (type default))
+  )
   (wire (pts (xy 421.64 260.35) (xy 425.45 260.35))
     (stroke (width 0) (type default))
@@
     (stroke (width 0) (type default))
   )
+  (wire (pts (xy 190.5 74.93) (xy 199.39 74.93))
+    (stroke (width 0) (type default))
+  )
   (wire (pts (xy 368.3 104.14) (xy 332.74 104.14))
     (stroke (width 0) (type default))
@@
     (stroke (width 0) (type default))
   )
+  (wire (pts (xy 182.88 82.55) (xy 199.39 82.55))
+    (stroke (width 0) (type default))
+  )
   (wire (pts (xy 228.6 273.05) (xy 232.41 273.05))
     (stroke (width 0) (type default))
@@
     (stroke (width 0) (type default))
   )
+  (wire (pts (xy 421.64 80.01) (xy 425.45 80.01))
+    (stroke (width 0) (type default))
+  )
   (wire (pts (xy 392.43 100.33) (xy 370.84 100.33))
     (stroke (width 0) (type default))
@@
     (stroke (width 0) (type default))
   )
-  (wire (pts (xy 199.39 85.09) (xy 180.34 85.09))
+  (wire (pts (xy 421.64 232.41) (xy 425.45 232.41))
     (stroke (width 0) (type default))
   )
@@
     (stroke (width 0) (type default))
   )
-  (wire (pts (xy 199.39 74.93) (xy 190.5 74.93))
-    (stroke (width 0) (type default))
-  )
   (wire (pts (xy 228.6 264.16) (xy 232.41 264.16))
     (stroke (width 0) (type default))
@@
     (stroke (width 0) (type default))
   )
-  (wire (pts (xy 199.39 87.63) (xy 177.8 87.63))
-    (stroke (width 0) (type default))
-  )
   (wire (pts (xy 228.6 257.81) (xy 232.41 257.81))
     (stroke (width 0) (type default))
@@
     (stroke (width 0) (type default))
   )
+  (wire (pts (xy 175.26 90.17) (xy 199.39 90.17))
+    (stroke (width 0) (type default))
+  )
   (wire (pts (xy 180.34 275.59) (xy 140.97 275.59))
     (stroke (width 0) (type default))
@@
     (stroke (width 0) (type default))
   )
-  (wire (pts (xy 199.39 77.47) (xy 187.96 77.47))
-    (stroke (width 0) (type default))
-  )
   (wire (pts (xy 199.39 102.87) (xy 180.34 102.87))
     (stroke (width 0) (type default))
@@
     (stroke (width 0) (type default))
   )
+  (wire (pts (xy 228.6 232.41) (xy 232.41 232.41))
+    (stroke (width 0) (type default))
+  )
   (wire (pts (xy 392.43 242.57) (xy 368.3 242.57))
     (stroke (width 0) (type default))
@@
     (stroke (width 0) (type default))
   )
+  (wire (pts (xy 180.34 85.09) (xy 199.39 85.09))
+    (stroke (width 0) (type default))
+  )
   (wire (pts (xy 199.39 97.79) (xy 175.26 97.79))
     (stroke (width 0) (type default))
@@
       )
       (project "Quartz_v1p1"
-        (path "/674e1e7f-67ba-4e85-a926-dcd5f6a22021/db3c7ba2-982f-432b-8742-662861d58c3e"
-          (reference "R26") (unit 1)
-        )
         (path "/674e1e7f-67ba-4e85-a926-dcd5f6a22021"
           (reference "R1") (unit 1)
@@
       )
       (project "Quartz_v1p1"
-        (path "/674e1e7f-67ba-4e85-a926-dcd5f6a22021/db3c7ba2-982f-432b-8742-662861d58c3e"
-          (reference "R26") (unit 1)
-        )
         (path "/674e1e7f-67ba-4e85-a926-dcd5f6a22021"
           (reference "R3") (unit 1)
@@
       )
       (project "Quartz_v1p1"
-        (path "/674e1e7f-67ba-4e85-a926-dcd5f6a22021/c1293333-1878-4cba-a3bd-0c7884de1f1a"
-          (reference "#PWR025") (unit 1)
-        )
         (path "/674e1e7f-67ba-4e85-a926-dcd5f6a22021"
           (reference "#PWR01") (unit 1)
@@
       )
       (project "Quartz_v1p1"
-        (path "/674e1e7f-67ba-4e85-a926-dcd5f6a22021/db3c7ba2-982f-432b-8742-662861d58c3e"
-          (reference "R26") (unit 1)
-        )
         (path "/674e1e7f-67ba-4e85-a926-dcd5f6a22021"
           (reference "R2") (unit 1)
@@
       )
       (project "Quartz_v1p1"
-        (path "/674e1e7f-67ba-4e85-a926-dcd5f6a22021/c1293333-1878-4cba-a3bd-0c7884de1f1a"
-          (reference "#PWR025") (unit 1)
-        )
         (path "/674e1e7f-67ba-4e85-a926-dcd5f6a22021"
           (reference "#PWR03") (unit 1)
@@
       )
       (project "Quartz_v1p1"
-        (path "/674e1e7f-67ba-4e85-a926-dcd5f6a22021/c1293333-1878-4cba-a3bd-0c7884de1f1a"
-          (reference "#PWR025") (unit 1)
-        )
         (path "/674e1e7f-67ba-4e85-a926-dcd5f6a22021"
           (reference "#PWR02") (unit 1)
@@
       (effects (font (size 1.27 1.27) (color 72 72 72 1)) (justify left))
     )
-    (pin "AIN2+" input (at 199.39 85.09 180)
+    (pin "AIN2+" input (at 199.39 80.01 180)
       (effects (font (size 1.27 1.27) (color 72 72 72 1)) (justify left))
     )
-    (pin "AIN3+" input (at 199.39 90.17 180)
+    (pin "AIN3+" input (at 199.39 74.93 180)
       (effects (font (size 1.27 1.27) (color 72 72 72 1)) (justify left))
     )
-    (pin "AIN2-" input (at 199.39 87.63 180)
+    (pin "AIN2-" input (at 199.39 82.55 180)
       (effects (font (size 1.27 1.27) (color 72 72 72 1)) (justify left))
     )
-    (pin "AIN3-" input (at 199.39 92.71 180)
+    (pin "AIN3-" input (at 199.39 77.47 180)
       (effects (font (size 1.27 1.27) (color 72 72 72 1)) (justify left))
     )
-    (pin "AIN0+" input (at 199.39 74.93 180)
+    (pin "AIN0+" input (at 199.39 90.17 180)
       (effects (font (size 1.27 1.27) (color 72 72 72 1)) (justify left))
     )
-    (pin "AIN0-" input (at 199.39 77.47 180)
+    (pin "AIN0-" input (at 199.39 92.71 180)
       (effects (font (size 1.27 1.27) (color 72 72 72 1)) (justify left))
     )
-    (pin "AIN1+" input (at 199.39 80.01 180)
+    (pin "AIN1+" input (at 199.39 85.09 180)
       (effects (font (size 1.27 1.27) (color 72 72 72 1)) (justify left))
     )
-    (pin "AIN1-" input (at 199.39 82.55 180)
+    (pin "AIN1-" input (at 199.39 87.63 180)
       (effects (font (size 1.27 1.27) (color 72 72 72 1)) (justify left))
     )
@@
   )
   (sheet_instances
-    (path "/" (page "50"))
+    (path "/" (page "0"))
   )
 )

Commit message: Updated Layout
-Additional Layout Work
Connections:
- no-connect marks 3 -> 13
Other:
- sheet Channel1 renamed Channel01
- sheet Channel2 renamed Channel02
- sheet Channel3 renamed Channel03
- sheet Channel4 renamed Channel04
- sheet Channel5 renamed Channel05
- sheet Channel6 renamed Channel06
- sheet Channel7 renamed Channel07
- sheet Channel8 renamed Channel08
- sheet Channel9 renamed Channel09
- sheet Channel05: file input_filter_channel_INA851.kicad_sch -> input_filter_channel_INA851_flipped.kicad_sch
- sheet Channel06: file input_filter_channel_INA851.kicad_sch -> input_filter_channel_INA851_flipped.kicad_sch
- sheet Channel07: file input_filter_channel_INA851.kicad_sch -> input_filter_channel_INA851_flipped.kicad_sch
- sheet Channel08: file input_filter_channel_INA851.kicad_sch -> input_filter_channel_INA851_flipped.kicad_sch
- sheet Channel13: file input_filter_channel_INA851.kicad_sch -> input_filter_channel_INA851_flipped.kicad_sch
- sheet Channel14: file input_filter_channel_INA851.kicad_sch -> input_filter_channel_INA851_flipped.kicad_sch
- sheet Channel15: file input_filter_channel_INA851.kicad_sch -> input_filter_channel_INA851_flipped.kicad_sch
- sheet Channel16: file input_filter_channel_INA851.kicad_sch -> input_filter_channel_INA851_flipped.kicad_sch
- sheet Channel21: file input_filter_channel_INA851.kicad_sch -> input_filter_channel_INA851_flipped.kicad_sch
- sheet Channel22: file input_filter_channel_INA851.kicad_sch -> input_filter_channel_INA851_flipped.kicad_sch
- sheet Channel23: file input_filter_channel_INA851.kicad_sch -> input_filter_channel_INA851_flipped.kicad_sch
- sheet Channel24: file input_filter_channel_INA851.kicad_sch -> input_filter_channel_INA851_flipped.kicad_sch
- sheet Channel29: file input_filter_channel_INA851.kicad_sch -> input_filter_channel_INA851_flipped.kicad_sch
- sheet Channel30: file input_filter_channel_INA851.kicad_sch -> input_filter_channel_INA851_flipped.kicad_sch
- sheet Channel31: file input_filter_channel_INA851.kicad_sch -> input_filter_channel_INA851_flipped.kicad_sch
- sheet Channel32: file input_filter_channel_INA851.kicad_sch -> input_filter_channel_INA851_flipped.kicad_sch

Commit message: Updated Project
Schematics:
-updated level shifting IC's
-Add notes to level shifters
-Changed Relay Coil Driver channel mapping
-Added additional Mounting Hole

Layout
-WIP To Complete:
-Relay Driver ICs
- Reworking LT8582 area
- Level Shifters
- Housekeeping ICs
-Misc. error cleanup
- Silkscreen adjust
- Add Silkscreen SN & logo
Connections:
- net VDD renamed VDD1P8V

Commit message: Updated Project with Latest Changes
Project:
-Added pdf plots of PCB layout

Schematics:
-Fixed L8 Pinout
-Adjusted FMC connections
-Adjusted level shifter connections

Layout:
-Completed AFE/ADC/Power/Relay driver sections

Layout WIP To Complete:
-Misc. error cleanup
- Silkscreen adjust
- Add Silkscreen SN & logo
Parts:
- R? (x3): footprint Resistor_SMD:R_0603_1608Metric -> Resistor_SMD:R_0402_1005Metric
Changed lines of the file:
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@@
     (stroke (width 0) (type default))
   )
+  (wire (pts (xy 140.97 163.83) (xy 168.91 163.83))
+    (stroke (width 0) (type default))
+  )
   (wire (pts (xy 332.74 101.6) (xy 365.76 101.6))
     (stroke (width 0) (type default))
@@
     (stroke (width 0) (type default))
   )
-  (wire (pts (xy 193.04 163.83) (xy 168.91 163.83))
-    (stroke (width 0) (type default))
-  )
   (wire (pts (xy 332.74 220.98) (xy 361.95 220.98))
     (stroke (width 0) (type default))
@@
     (stroke (width 0) (type default))
   )
+  (wire (pts (xy 168.91 163.83) (xy 193.04 163.83))
+    (stroke (width 0) (type default))
+  )
   (wire (pts (xy 140.97 72.39) (xy 161.29 72.39))
     (stroke (width 0) (type default))
@@
     (stroke (width 0) (type default))
   )
-  (wire (pts (xy 168.91 163.83) (xy 140.97 163.83))
-    (stroke (width 0) (type default))
-  )
   (wire (pts (xy 361.95 144.78) (xy 361.95 163.83))
     (stroke (width 0) (type default))
@@
     (effects (font (size 1.27 1.27)) (justify left bottom))
   )
+  (label "ADC_VCM4" (at 374.65 316.23 0) (fields_autoplaced)
+    (effects (font (size 1.27 1.27)) (justify left bottom))
+  )
+  (label "ADC_VCM1" (at 180.975 163.83 0) (fields_autoplaced)
+    (effects (font (size 1.27 1.27)) (justify left bottom))
+  )
   (label "AIN26+" (at 283.21 90.17 0) (fields_autoplaced)
     (effects (font (size 1.27 1.27)) (justify left bottom))
@@
     (effects (font (size 1.27 1.27)) (justify left bottom))
   )
+  (label "ADC_VCM3" (at 374.65 163.83 0) (fields_autoplaced)
+    (effects (font (size 1.27 1.27)) (justify left bottom))
+  )
   (label "AIN9+" (at 91.44 86.36 0) (fields_autoplaced)
     (effects (font (size 1.27 1.27)) (justify left bottom))
@@
     (effects (font (size 1.27 1.27)) (justify left bottom))
   )
+  (label "ADC_VCM2" (at 181.61 316.23 0) (fields_autoplaced)
+    (effects (font (size 1.27 1.27)) (justify left bottom))
+  )
   (label "Relay_ResetCoil32" (at 334.01 322.58 0) (fields_autoplaced)
     (effects (font (size 1.27 1.27)) (justify left bottom))
@@
       (effects (font (size 1.27 1.27)) (justify left))
     )
-    (property "Footprint" "Resistor_SMD:R_0603_1608Metric" (at 232.41 220.98 0)
+    (property "Footprint" "Resistor_SMD:R_0402_1005Metric" (at 232.41 220.98 0)
       (effects (font (size 1.27 1.27)) hide)
     )
@@
       (effects (font (size 1.27 1.27)) (justify left))
     )
-    (property "Footprint" "Resistor_SMD:R_0603_1608Metric" (at 425.45 220.98 0)
+    (property "Footprint" "Resistor_SMD:R_0402_1005Metric" (at 425.45 220.98 0)
       (effects (font (size 1.27 1.27)) hide)
     )
@@
       (effects (font (size 1.27 1.27)) (justify left))
     )
-    (property "Footprint" "Resistor_SMD:R_0603_1608Metric" (at 425.45 68.58 0)
+    (property "Footprint" "Resistor_SMD:R_0402_1005Metric" (at 425.45 68.58 0)
       (effects (font (size 1.27 1.27)) hide)
     )
@@
   )
   (sheet_instances
-    (path "/" (page "50"))
+    (path "/" (page "0"))
   )
 )

Commit message: Push Version before ADC change from 1.8V to 2.5V I/O
Changed lines of the file:
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@@
     (stroke (width 0) (type default))
   )
-  (bus_entry (at 162.56 153.67) (size -2.54 -2.54)
-    (stroke (width 0) (type default))
-  )
   (bus_entry (at 353.06 167.64) (size 2.54 2.54)
     (stroke (width 0) (type default))
@@
     (stroke (width 0) (type default))
   )
+  (bus_entry (at 160.02 151.13) (size 2.54 2.54)
+    (stroke (width 0) (type default))
+  )
   (bus_entry (at 354.33 287.02) (size -2.54 -2.54)
     (stroke (width 0) (type default))
@@
     (stroke (width 0) (type default))
   )
-  (wire (pts (xy 161.29 167.64) (xy 140.97 167.64))
+  (wire (pts (xy 140.97 167.64) (xy 161.29 167.64))
     (stroke (width 0) (type default))
   )
@@
   )
   (sheet_instances
-    (path "/" (page "0"))
+    (path "/" (page "50"))
   )
 )

Commit message: Changed ADCs to run on +2.5V VADJ
Modified schematic to allow the ADCs to be run from the +2.5V VADJ inputs on the FMC connector.
-All relevant ERC issues ran been looked into.
-Still working on all Board DRC issues.
Connections:
- net VDD1P8V renamed P2_VADJ
- net P2_VADJ: no longer R?.1
- new net P1_VADJ: R?.1
Other:
- sheet ADC3: file ADC.kicad_sch -> ADC_P2.kicad_sch
- sheet ADC4: file ADC.kicad_sch -> ADC_P2.kicad_sch
- note added: "+2.5V"
Changed lines of the file:
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@@
     (stroke (width 0) (type default))
+  )
+  (text "+2.5V" (at 429.895 217.805 0)
+    (effects (font (size 1.27 1.27)) (justify left bottom))
+  )
+  (text "+2.5V" (at 429.895 65.405 0)
+    (effects (font (size 1.27 1.27)) (justify left bottom))
+  )
+  (text "+2.5V" (at 236.855 217.805 0)
+    (effects (font (size 1.27 1.27)) (justify left bottom))
   )
   (label "Relay_ResetCoil4" (at 142.24 93.98 0) (fields_autoplaced)
@@
     )
   )
+  (global_label "P1_VADJ" (shape input) (at 232.41 214.63 0) (fields_autoplaced)
+    (effects (font (size 1.27 1.27)) (justify left))
+    (property "Intersheetrefs" "${INTERSHEET_REFS}" (at 243.1777 214.63 0)
+      (effects (font (size 1.27 1.27)) (justify left) hide)
+    )
+  )
   (global_label "ADC2_MCLK+" (shape input) (at 232.41 273.05 0) (fields_autoplaced)
     (effects (font (size 1.27 1.27)) (justify left))
@@
     )
   )
+  (global_label "P2_VADJ" (shape input) (at 425.45 214.63 0) (fields_autoplaced)
+    (effects (font (size 1.27 1.27)) (justify left))
+    (property "Intersheetrefs" "${INTERSHEET_REFS}" (at 436.2177 214.63 0)
+      (effects (font (size 1.27 1.27)) (justify left) hide)
+    )
+  )
   (global_label "AD7768_SCLK" (shape input) (at 425.45 266.7 0) (fields_autoplaced)
     (effects (font (size 1.27 1.27)) (justify left))
@@
     )
   )
-  (global_label "VDD1P8V" (shape input) (at 425.45 62.23 0) (fields_autoplaced)
-    (effects (font (size 1.27 1.27)) (justify left))
-    (property "Intersheetrefs" "${INTERSHEET_REFS}" (at 436.762 62.23 0)
-      (effects (font (size 1.27 1.27)) (justify left) hide)
-    )
-  )
   (global_label "ADC1_SDO" (shape input) (at 232.41 116.84 0) (fields_autoplaced)
     (effects (font (size 1.27 1.27)) (justify left))
@@
     )
   )
-  (global_label "VDD1P8V" (shape input) (at 425.45 214.63 0) (fields_autoplaced)
-    (effects (font (size 1.27 1.27)) (justify left))
-    (property "Intersheetrefs" "${INTERSHEET_REFS}" (at 436.762 214.63 0)
-      (effects (font (size 1.27 1.27)) (justify left) hide)
-    )
-  )
   (global_label "ADC3_DO1" (shape input) (at 425.45 90.17 0) (fields_autoplaced)
     (effects (font (size 1.27 1.27)) (justify left))
@@
     )
   )
+  (global_label "P2_VADJ" (shape input) (at 425.45 62.23 0) (fields_autoplaced)
+    (effects (font (size 1.27 1.27)) (justify left))
+    (property "Intersheetrefs" "${INTERSHEET_REFS}" (at 436.2177 62.23 0)
+      (effects (font (size 1.27 1.27)) (justify left) hide)
+    )
+  )
   (global_label "ADC2_DO6" (shape input) (at 232.41 255.27 0) (fields_autoplaced)
     (effects (font (size 1.27 1.27)) (justify left))
@@
     (effects (font (size 1.27 1.27)) (justify left))
     (property "Intersheetrefs" "${INTERSHEET_REFS}" (at 440.8328 275.59 0)
-      (effects (font (size 1.27 1.27)) (justify left) hide)
-    )
-  )
-  (global_label "VDD1P8V" (shape input) (at 232.41 214.63 0) (fields_autoplaced)
-    (effects (font (size 1.27 1.27)) (justify left))
-    (property "Intersheetrefs" "${INTERSHEET_REFS}" (at 243.722 214.63 0)
       (effects (font (size 1.27 1.27)) (justify left) hide)
     )
@@
       (effects (font (size 1.27 1.27)) (justify left bottom))
     )
-    (property "Sheetfile" "ADC.kicad_sch" (at 392.43 126.3146 0)
+    (property "Sheetfile" "ADC_P2.kicad_sch" (at 392.43 126.3146 0)
       (effects (font (size 1.27 1.27)) (justify left top))
     )
@@
       (effects (font (size 1.27 1.27)) (justify left bottom))
     )
-    (property "Sheetfile" "ADC.kicad_sch" (at 392.43 278.7146 0)
+    (property "Sheetfile" "ADC_P2.kicad_sch" (at 392.43 278.7146 0)
       (effects (font (size 1.27 1.27)) (justify left top))
     )

Commit message: Completed Schmatic and Layout
All Schematic and Layout Task are complete with the following exceptions:
- Adjust Silkscreen Layers
- Add Osprey Logo and Serial Number

Note-Removed Files no longer reference in the project
Parts:
- removed R? (x3): 4.75k, Resistor_SMD:R_0402_1005Metric, symbol Device:R_Small_US
- added R? (x3): 4.75k, Resistor_SMD:R_0402_1005Metric, symbol Device:R_Small_US
- J1, J2: symbol Connector:DC37_Receptacle -> AD7768_Digitizer_SLib:DC37_Receptacle
Connections:
- net ADC2/ADC_~{Start}: now also R?.1
- net ADC3/ADC_~{Start}: now also R?.1
- net ADC4/ADC_~{Start}: now also R?.1
- new net GND: J1.38, J1.39, J2.38, J2.39
- new net P1_2P5V: R?.2
- new net P2_2P5V: R?.2, R?.2
Other:
- sheet ADC1 ports: added AD7768_SDI, AD7768_~{RESET}, IOVDD; removed none
- sheet ADC2 ports: added AD7768_SDI, AD7768_~{RESET}, IOVDD; removed none
- sheet ADC3: file ADC_P2.kicad_sch -> ADC.kicad_sch
- sheet ADC3 ports: added AD7768_SDI, AD7768_~{RESET}, IOVDD; removed none
- sheet ADC4: file ADC_P2.kicad_sch -> ADC.kicad_sch
- sheet ADC4 ports: added AD7768_SDI, AD7768_~{RESET}, IOVDD; removed none
- sheet Channel05: file input_filter_channel_INA851_flipped.kicad_sch -> input_filter_channel_INA851.kicad_sch
- sheet Channel06: file input_filter_channel_INA851_flipped.kicad_sch -> input_filter_channel_INA851.kicad_sch
- sheet Channel07: file input_filter_channel_INA851_flipped.kicad_sch -> input_filter_channel_INA851.kicad_sch
- sheet Channel08: file input_filter_channel_INA851_flipped.kicad_sch -> input_filter_channel_INA851.kicad_sch
- sheet Channel13: file input_filter_channel_INA851_flipped.kicad_sch -> input_filter_channel_INA851.kicad_sch
- sheet Channel14: file input_filter_channel_INA851_flipped.kicad_sch -> input_filter_channel_INA851.kicad_sch
- sheet Channel15: file input_filter_channel_INA851_flipped.kicad_sch -> input_filter_channel_INA851.kicad_sch
- sheet Channel16: file input_filter_channel_INA851_flipped.kicad_sch -> input_filter_channel_INA851.kicad_sch
- sheet Channel21: file input_filter_channel_INA851_flipped.kicad_sch -> input_filter_channel_INA851.kicad_sch
- sheet Channel22: file input_filter_channel_INA851_flipped.kicad_sch -> input_filter_channel_INA851.kicad_sch
- sheet Channel23: file input_filter_channel_INA851_flipped.kicad_sch -> input_filter_channel_INA851.kicad_sch
- sheet Channel24: file input_filter_channel_INA851_flipped.kicad_sch -> input_filter_channel_INA851.kicad_sch
- sheet Channel29: file input_filter_channel_INA851_flipped.kicad_sch -> input_filter_channel_INA851.kicad_sch
- sheet Channel30: file input_filter_channel_INA851_flipped.kicad_sch -> input_filter_channel_INA851.kicad_sch
- sheet Channel31: file input_filter_channel_INA851_flipped.kicad_sch -> input_filter_channel_INA851.kicad_sch
- sheet Channel32: file input_filter_channel_INA851_flipped.kicad_sch -> input_filter_channel_INA851.kicad_sch
- note removed: "+2.5V"
