File: Quartz_v1p1.kicad_sch (KiCad schematic)
At the start: 13 parts, among them J1 DB37, J2 DB37

Commit message: Updates to Design
-Flipped D10 to correct side of board
-Moved and verified mounting hole position
- Fixed PNs for R1,R2,R3 and LT8582 part
-added configurable grounding for DB37 center pins
Parts:
- added R116, R117, R71, R72: DNI, Resistor_SMD:R_0805_2012Metric, symbol Device:R_Small_US
- R? (x3): MPN RC0603FR-074K75L -> RC0402FR-074K75L
Connections:
- net Earth: now also R116.1, R71.1
- net GND: now also R117.1, R72.1
- net at J2.10: now also J2.11, J2.28, J2.29, J2.9, R116.2, R117.2
- net at J1.10: now also J1.11, J1.28, J1.29, J1.9, R71.2, R72.2
- no-connect marks 13 -> 3
Other:
- moved on the sheet: J1, J2, R?
