File: input_filter_channel_INA851.kicad_sch (KiCad schematic)
At the start: 28 parts, among them K1 EE2-12TNU-L, U101 INA851

Commit message: Updated Project with Latest Changes
Project:
-Added pdf plots of PCB layout

Schematics:
-Fixed L8 Pinout
-Adjusted FMC connections
-Adjusted level shifter connections

Layout:
-Completed AFE/ADC/Power/Relay driver sections

Layout WIP To Complete:
-Misc. error cleanup
- Silkscreen adjust
- Add Silkscreen SN & logo
Parts:
- U101: footprint Package_DFN_QFN:QFN-16-1EP_3x3mm_P0.5mm_EP1.75x1.75mm_ThermalVias -> footprints:QFN-16-1EP_3x3mm_P0.5mm_EP1.75x1.75mm_ThermalVias
Changed lines of the file:
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@@
       (effects (font (size 1.27 1.27)))
     )
-    (property "Footprint" "Package_DFN_QFN:QFN-16-1EP_3x3mm_P0.5mm_EP1.75x1.75mm_ThermalVias" (at 147.32 77.47 0)
+    (property "Footprint" "footprints:QFN-16-1EP_3x3mm_P0.5mm_EP1.75x1.75mm_ThermalVias" (at 147.32 77.47 0)
       (effects (font (size 1.27 1.27)) hide)
     )

Commit message: Updated PCB
Adjusted Silkscreen
Added Logo and SN location
Parts:
- C? (x3): MPN 0603N820J500CT -> DNI
- C? (x2): MPN 0603N820J500CT -> CC0402JRNPO9BN820
- C?: MPN GCM1885C1H101JA16D -> GRM1885C1H101JA01D
- C? (x3): MPN CL10B104KB8NNWC -> CL05A104KA5NNNC
- C?: MPN (none) -> GRT155R61C474KE01D
- K1: footprint Relay_SMD:Relay_DPDT_Kemet_EE2_NU_DoubleCoil -> footprints:Relay_DPDT_Kemet_EE2_NU_DoubleCoil
- R?: MPN (none) -> DNI
- R? (x4): MPN ERJ-3GEY0R00V -> ERJ-2GE0R00X
- R? (x2): MPN RC0603FR-0782RL -> RC0402FR-0782RL
Changed lines of the file:
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@@
       (effects (font (size 1.27 1.27)) hide)
     )
-    (property "MPN" "0603N820J500CT" (at 119.38 90.17 0)
+    (property "MPN" "DNI" (at 119.38 90.17 0)
       (effects (font (size 1.27 1.27)) hide)
     )
@@
       (effects (font (size 1.27 1.27)) hide)
     )
-    (property "MPN" "0603N820J500CT" (at 213.36 97.79 0)
+    (property "MPN" "CC0402JRNPO9BN820" (at 213.36 97.79 0)
       (effects (font (size 1.27 1.27)) hide)
     )
@@
       (effects (font (size 1.27 1.27)) hide)
     )
-    (property "MPN" "" (at 142.24 91.44 90)
+    (property "MPN" "DNI" (at 142.24 91.44 90)
       (effects (font (size 1.27 1.27)) hide)
     )
@@
       (effects (font (size 1.27 1.27)) hide)
     )
-    (property "MPN" "ERJ-3GEY0R00V" (at 176.53 97.79 90)
+    (property "MPN" "ERJ-2GE0R00X" (at 176.53 97.79 90)
       (effects (font (size 1.27 1.27)) hide)
     )
@@
       (effects (font (size 1.27 1.27)) hide)
     )
-    (property "MPN" "GCM1885C1H101JA16D" (at 227.33 92.71 0)
+    (property "MPN" "GRM1885C1H101JA01D" (at 227.33 92.71 0)
       (effects (font (size 1.27 1.27)) hide)
     )
@@
       (effects (font (size 1.27 1.27)) hide)
     )
-    (property "MPN" "ERJ-3GEY0R00V" (at 177.8 86.36 90)
+    (property "MPN" "ERJ-2GE0R00X" (at 177.8 86.36 90)
       (effects (font (size 1.27 1.27)) hide)
     )
@@
       (effects (font (size 1.27 1.27)) hide)
     )
-    (property "MPN" "CL10B104KB8NNWC" (at 189.23 72.39 0)
+    (property "MPN" "CL05A104KA5NNNC" (at 189.23 72.39 0)
       (effects (font (size 1.27 1.27)) hide)
     )
@@
       (effects (font (size 1.27 1.27)) hide)
     )
-    (property "MPN" "0603N820J500CT" (at 213.36 88.9 0)
+    (property "MPN" "CC0402JRNPO9BN820" (at 213.36 88.9 0)
       (effects (font (size 1.27 1.27)) hide)
     )
@@
       (effects (font (size 1.27 1.27)) hide)
     )
-    (property "MPN" "CL10B104KB8NNWC" (at 162.56 67.31 0)
+    (property "MPN" "CL05A104KA5NNNC" (at 162.56 67.31 0)
       (effects (font (size 1.27 1.27)) hide)
     )
@@
       (effects (font (size 1.27 1.27)) hide)
     )
-    (property "MPN" "" (at 168.91 120.65 0)
+    (property "MPN" "GRT155R61C474KE01D" (at 168.91 120.65 0)
       (effects (font (size 1.27 1.27)) hide)
     )
@@
       (effects (font (size 1.27 1.27)) hide)
     )
-    (property "MPN" "0603N820J500CT" (at 107.95 93.98 0)
+    (property "MPN" "DNI" (at 107.95 93.98 0)
       (effects (font (size 1.27 1.27)) hide)
     )
@@
       (effects (font (size 1.27 1.27)) hide)
     )
-    (property "MPN" "ERJ-3GEY0R00V" (at 99.06 86.36 90)
+    (property "MPN" "ERJ-2GE0R00X" (at 99.06 86.36 90)
       (effects (font (size 1.27 1.27)) hide)
     )
@@
       (effects (font (size 1.27 1.27)) hide)
     )
-    (property "MPN" "CL10B104KB8NNWC" (at 149.86 118.745 0)
+    (property "MPN" "CL05A104KA5NNNC" (at 149.86 118.745 0)
       (effects (font (size 1.27 1.27)) hide)
     )
@@
       (effects (font (size 1.27 1.27)) hide)
     )
-    (property "MPN" "0603N820J500CT" (at 107.95 88.9 0)
+    (property "MPN" "DNI" (at 107.95 88.9 0)
       (effects (font (size 1.27 1.27)) hide)
     )
@@
       (effects (font (size 1.27 1.27)) hide)
     )
-    (property "MPN" "RC0603FR-0782RL" (at 195.58 90.17 90)
+    (property "MPN" "RC0402FR-0782RL" (at 195.58 90.17 90)
       (effects (font (size 1.27 1.27)) hide)
     )
@@
       (effects (font (size 1.27 1.27)) hide)
     )
-    (property "MPN" "RC0603FR-0782RL" (at 195.58 93.98 90)
+    (property "MPN" "RC0402FR-0782RL" (at 195.58 93.98 90)
       (effects (font (size 1.27 1.27)) hide)
     )
@@
       (effects (font (size 1.27 1.27)) hide)
     )
-    (property "MPN" "ERJ-3GEY0R00V" (at 99.06 96.52 90)
+    (property "MPN" "ERJ-2GE0R00X" (at 99.06 96.52 90)
       (effects (font (size 1.27 1.27)) hide)
     )
@@
       (effects (font (size 1.27 1.27)))
     )
-    (property "Footprint" "Relay_SMD:Relay_DPDT_Kemet_EE2_NU_DoubleCoil" (at 80.01 96.52 0)
+    (property "Footprint" "footprints:Relay_DPDT_Kemet_EE2_NU_DoubleCoil" (at 80.01 96.52 0)
       (effects (font (size 1.27 1.27)) hide)
     )

Commit message: Finalized Design & Board
Change to design
-Added resistor options to choose the grounding of input connectors
-uploaded libraries
-uploaded generated BOM
- adjusted mounting holes on front of board by 10mil
-Changed input AC blocking cap to 10nF from 100nF due to part availability
Parts:
- C? (x2): value 100nF -> 10nF
- C? (x3): now left out of the parts list
- K1: footprint footprints:Relay_DPDT_Kemet_EE2_NU_DoubleCoil -> QuartzFootprints:Relay_DPDT_Kemet_EE2_NU_DoubleCoil
- R?: value open -> DNI; now left out of the parts list
- U101: footprint footprints:QFN-16-1EP_3x3mm_P0.5mm_EP1.75x1.75mm_ThermalVias -> QuartzFootprints:QFN-16-1EP_3x3mm_P0.5mm_EP1.75x1.75mm_ThermalVias
Changed lines of the file:
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@@
       (effects (font (size 1.27 1.27)) (justify left))
     )
-    (property "Value" "100nF" (at 73.66 97.79 90)
+    (property "Value" "10nF" (at 73.66 97.79 90)
       (effects (font (size 1.27 1.27)) (justify left))
     )
@@
   )
   (symbol (lib_id "Device:C_Small") (at 119.38 90.17 0) (unit 1)
-    (in_bom yes) (on_board yes) (dnp yes)
+    (in_bom no) (on_board yes) (dnp yes)
     (property "Reference" "C?" (at 121.92 89.5413 0)
       (effects (font (size 1.27 1.27)) (justify left))
@@
   )
   (symbol (lib_id "Device:R_Small_US") (at 142.24 91.44 0) (unit 1)
-    (in_bom yes) (on_board yes) (dnp yes)
+    (in_bom no) (on_board yes) (dnp yes)
     (property "Reference" "R?" (at 138.43 92.71 0)
       (effects (font (size 1.27 1.27)))
     )
-    (property "Value" "open" (at 140.97 90.17 0)
+    (property "Value" "DNI" (at 140.97 90.17 0)
       (effects (font (size 1.27 1.27)) (justify right))
     )
@@
       (effects (font (size 1.27 1.27)))
     )
-    (property "Footprint" "footprints:QFN-16-1EP_3x3mm_P0.5mm_EP1.75x1.75mm_ThermalVias" (at 147.32 77.47 0)
+    (property "Footprint" "QuartzFootprints:QFN-16-1EP_3x3mm_P0.5mm_EP1.75x1.75mm_ThermalVias" (at 147.32 77.47 0)
       (effects (font (size 1.27 1.27)) hide)
     )
@@
   )
   (symbol (lib_id "Device:C_Small") (at 107.95 93.98 0) (unit 1)
-    (in_bom yes) (on_board yes) (dnp yes)
+    (in_bom no) (on_board yes) (dnp yes)
     (property "Reference" "C?" (at 110.49 93.3513 0)
       (effects (font (size 1.27 1.27)) (justify left))
@@
   )
   (symbol (lib_id "Device:C_Small") (at 107.95 88.9 0) (unit 1)
-    (in_bom yes) (on_board yes) (dnp yes)
+    (in_bom no) (on_board yes) (dnp yes)
     (property "Reference" "C?" (at 110.49 88.2713 0)
       (effects (font (size 1.27 1.27)) (justify left))
@@
       (effects (font (size 1.27 1.27)))
     )
-    (property "Footprint" "footprints:Relay_DPDT_Kemet_EE2_NU_DoubleCoil" (at 80.01 96.52 0)
+    (property "Footprint" "QuartzFootprints:Relay_DPDT_Kemet_EE2_NU_DoubleCoil" (at 80.01 96.52 0)
       (effects (font (size 1.27 1.27)) hide)
     )
@@
       (effects (font (size 1.27 1.27)) (justify left))
     )
-    (property "Value" "100nF" (at 73.66 90.17 90)
+    (property "Value" "10nF" (at 73.66 90.17 90)
       (effects (font (size 1.27 1.27)) (justify left))
     )

Commit message: Updated with all Quartz v1.2 changes
-Fixed issue with pinouts on current sense chip and Mosfet on 15V split rail section
-moved DB37 connectors by 30mil for front panel alignment
- Added 12V test point
Parts:
- R?: MPN DNI -> TNPW040211K8BEED; now fitted; now in the parts list
Changed lines of the file:
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@@
         )
       )
-      (project "Quartz_v1p1"
+      (project "Quartz_v1p2"
         (path "/674e1e7f-67ba-4e85-a926-dcd5f6a22021/40baf21a-c5b6-4126-86f5-a663d00e8f52"
           (reference "C102") (unit 1)
@@
         )
       )
-      (project "Quartz_v1p1"
+      (project "Quartz_v1p2"
         (path "/674e1e7f-67ba-4e85-a926-dcd5f6a22021/40baf21a-c5b6-4126-86f5-a663d00e8f52"
           (reference "#PWR0107") (unit 1)
@@
         )
       )
-      (project "Quartz_v1p1"
+      (project "Quartz_v1p2"
         (path "/674e1e7f-67ba-4e85-a926-dcd5f6a22021/40baf21a-c5b6-4126-86f5-a663d00e8f52"
           (reference "#PWR0108") (unit 1)
@@
         )
       )
-      (project "Quartz_v1p1"
+      (project "Quartz_v1p2"
         (path "/674e1e7f-67ba-4e85-a926-dcd5f6a22021/40baf21a-c5b6-4126-86f5-a663d00e8f52"
           (reference "C105") (unit 1)
@@
         )
       )
-      (project "Quartz_v1p1"
+      (project "Quartz_v1p2"
         (path "/674e1e7f-67ba-4e85-a926-dcd5f6a22021/40baf21a-c5b6-4126-86f5-a663d00e8f52"
           (reference "R103") (unit 1)
@@
         )
       )
-      (project "Quartz_v1p1"
+      (project "Quartz_v1p2"
         (path "/674e1e7f-67ba-4e85-a926-dcd5f6a22021/40baf21a-c5b6-4126-86f5-a663d00e8f52"
           (reference "C112") (unit 1)
@@
         )
       )
-      (project "Quartz_v1p1"
+      (project "Quartz_v1p2"
         (path "/674e1e7f-67ba-4e85-a926-dcd5f6a22021/40baf21a-c5b6-4126-86f5-a663d00e8f52"
           (reference "#PWR0106") (unit 1)
@@
   )
   (symbol (lib_id "Device:R_Small_US") (at 142.24 91.44 0) (unit 1)
-    (in_bom no) (on_board yes) (dnp yes)
+    (in_bom yes) (on_board yes) (dnp no)
     (property "Reference" "R?" (at 138.43 92.71 0)
       (effects (font (size 1.27 1.27)))
@@
       (effects (font (size 1.27 1.27)) hide)
     )
-    (property "MPN" "DNI" (at 142.24 91.44 90)
+    (property "MPN" "TNPW040211K8BEED" (at 142.24 91.44 90)
       (effects (font (size 1.27 1.27)) hide)
     )
@@
         )
       )
-      (project "Quartz_v1p1"
+      (project "Quartz_v1p2"
         (path "/674e1e7f-67ba-4e85-a926-dcd5f6a22021/40baf21a-c5b6-4126-86f5-a663d00e8f52"
           (reference "R105") (unit 1)
@@
         )
       )
-      (project "Quartz_v1p1"
+      (project "Quartz_v1p2"
         (path "/674e1e7f-67ba-4e85-a926-dcd5f6a22021/40baf21a-c5b6-4126-86f5-a663d00e8f52"
           (reference "R106") (unit 1)
@@
         )
       )
-      (project "Quartz_v1p1"
+      (project "Quartz_v1p2"
         (path "/674e1e7f-67ba-4e85-a926-dcd5f6a22021/40baf21a-c5b6-4126-86f5-a663d00e8f52"
           (reference "C113") (unit 1)
@@
         )
       )
-      (project "Quartz_v1p1"
+      (project "Quartz_v1p2"
         (path "/674e1e7f-67ba-4e85-a926-dcd5f6a22021/40baf21a-c5b6-4126-86f5-a663d00e8f52"
           (reference "R107") (unit 1)
@@
         )
       )
-      (project "Quartz_v1p1"
+      (project "Quartz_v1p2"
         (path "/674e1e7f-67ba-4e85-a926-dcd5f6a22021/40baf21a-c5b6-4126-86f5-a663d00e8f52"
           (reference "C110") (unit 1)
@@
         )
       )
-      (project "Quartz_v1p1"
+      (project "Quartz_v1p2"
         (path "/674e1e7f-67ba-4e85-a926-dcd5f6a22021/40baf21a-c5b6-4126-86f5-a663d00e8f52"
           (reference "#PWR0132") (unit 1)
@@
         )
       )
-      (project "Quartz_v1p1"
+      (project "Quartz_v1p2"
         (path "/674e1e7f-67ba-4e85-a926-dcd5f6a22021/40baf21a-c5b6-4126-86f5-a663d00e8f52"
           (reference "#PWR0111") (unit 1)
@@
     (pin "9")
     (instances
-      (project "Quartz_v1p1"
+      (project "Quartz_v1p2"
         (path "/674e1e7f-67ba-4e85-a926-dcd5f6a22021/40baf21a-c5b6-4126-86f5-a663d00e8f52"
           (reference "U101") (unit 1)
@@
         )
       )
-      (project "Quartz_v1p1"
+      (project "Quartz_v1p2"
         (path "/674e1e7f-67ba-4e85-a926-dcd5f6a22021/40baf21a-c5b6-4126-86f5-a663d00e8f52"
           (reference "#PWR0109") (unit 1)
@@
         )
       )
-      (project "Quartz_v1p1"
+      (project "Quartz_v1p2"
         (path "/674e1e7f-67ba-4e85-a926-dcd5f6a22021/40baf21a-c5b6-4126-86f5-a663d00e8f52"
           (reference "C119") (unit 1)
@@
     (pin "2")
     (instances
-      (project "Quartz_v1p1"
+      (project "Quartz_v1p2"
         (path "/674e1e7f-67ba-4e85-a926-dcd5f6a22021/40baf21a-c5b6-4126-86f5-a663d00e8f52"
           (reference "L101") (unit 1)
@@
         )
       )
-      (project "Quartz_v1p1"
+      (project "Quartz_v1p2"
         (path "/674e1e7f-67ba-4e85-a926-dcd5f6a22021/40baf21a-c5b6-4126-86f5-a663d00e8f52"
           (reference "C111") (unit 1)
@@
         )
       )
-      (project "Quartz_v1p1"
+      (project "Quartz_v1p2"
         (path "/674e1e7f-67ba-4e85-a926-dcd5f6a22021/40baf21a-c5b6-4126-86f5-a663d00e8f52"
           (reference "C109") (unit 1)
@@
         )
       )
-      (project "Quartz_v1p1"
+      (project "Quartz_v1p2"
         (path "/674e1e7f-67ba-4e85-a926-dcd5f6a22021/40baf21a-c5b6-4126-86f5-a663d00e8f52"
           (reference "C107") (unit 1)
@@
         )
       )
-      (project "Quartz_v1p1"
+      (project "Quartz_v1p2"
         (path "/674e1e7f-67ba-4e85-a926-dcd5f6a22021/40baf21a-c5b6-4126-86f5-a663d00e8f52"
           (reference "C108") (unit 1)
@@
         )
       )
-      (project "Quartz_v1p1"
+      (project "Quartz_v1p2"
         (path "/674e1e7f-67ba-4e85-a926-dcd5f6a22021/40baf21a-c5b6-4126-86f5-a663d00e8f52"
           (reference "C104") (unit 1)
@@
     (pin "2")
     (instances
-      (project "Quartz_v1p1"
+      (project "Quartz_v1p2"
         (path "/674e1e7f-67ba-4e85-a926-dcd5f6a22021/40baf21a-c5b6-4126-86f5-a663d00e8f52"
           (reference "L103") (unit 1)
@@
         )
       )
-      (project "Quartz_v1p1"
+      (project "Quartz_v1p2"
         (path "/674e1e7f-67ba-4e85-a926-dcd5f6a22021/40baf21a-c5b6-4126-86f5-a663d00e8f52"
           (reference "R101") (unit 1)
@@
         )
       )
-      (project "Quartz_v1p1"
+      (project "Quartz_v1p2"
         (path "/674e1e7f-67ba-4e85-a926-dcd5f6a22021/40baf21a-c5b6-4126-86f5-a663d00e8f52"
           (reference "#PWR0103") (unit 1)
@@
     (pin "2")
     (instances
-      (project "Quartz_v1p1"
+      (project "Quartz_v1p2"
         (path "/674e1e7f-67ba-4e85-a926-dcd5f6a22021/40baf21a-c5b6-4126-86f5-a663d00e8f52"
           (reference "L102") (unit 1)
@@
         )
       )
-      (project "Quartz_v1p1"
+      (project "Quartz_v1p2"
         (path "/674e1e7f-67ba-4e85-a926-dcd5f6a22021/40baf21a-c5b6-4126-86f5-a663d00e8f52"
           (reference "C106") (unit 1)
@@
         )
       )
-      (project "Quartz_v1p1"
+      (project "Quartz_v1p2"
         (path "/674e1e7f-67ba-4e85-a926-dcd5f6a22021/40baf21a-c5b6-4126-86f5-a663d00e8f52"
           (reference "#PWR0104") (unit 1)
@@
         )
       )
-      (project "Quartz_v1p1"
+      (project "Quartz_v1p2"
         (path "/674e1e7f-67ba-4e85-a926-dcd5f6a22021/40baf21a-c5b6-4126-86f5-a663d00e8f52"
           (reference "#PWR0105") (unit 1)
@@
         )
       )
-      (project "Quartz_v1p1"
+      (project "Quartz_v1p2"
         (path "/674e1e7f-67ba-4e85-a926-dcd5f6a22021/40baf21a-c5b6-4126-86f5-a663d00e8f52"
           (reference "C103") (unit 1)
@@
         )
       )
-      (project "Quartz_v1p1"
+      (project "Quartz_v1p2"
         (path "/674e1e7f-67ba-4e85-a926-dcd5f6a22021/40baf21a-c5b6-4126-86f5-a663d00e8f52"
           (reference "R108") (unit 1)
@@
         )
       )
-      (project "Quartz_v1p1"
+      (project "Quartz_v1p2"
         (path "/674e1e7f-67ba-4e85-a926-dcd5f6a22021/40baf21a-c5b6-4126-86f5-a663d00e8f52"
           (reference "R104") (unit 1)
@@
         )
       )
-      (project "Quartz_v1p1"
+      (project "Quartz_v1p2"
         (path "/674e1e7f-67ba-4e85-a926-dcd5f6a22021/40baf21a-c5b6-4126-86f5-a663d00e8f52"
           (reference "R109") (unit 1)
@@
         )
       )
-      (project "Quartz_v1p1"
+      (project "Quartz_v1p2"
         (path "/674e1e7f-67ba-4e85-a926-dcd5f6a22021/40baf21a-c5b6-4126-86f5-a663d00e8f52"
           (reference "R102") (unit 1)
@@
         )
       )
-      (project "Quartz_v1p1"
+      (project "Quartz_v1p2"
         (path "/674e1e7f-67ba-4e85-a926-dcd5f6a22021/40baf21a-c5b6-4126-86f5-a663d00e8f52"
           (reference "K101") (unit 1)
@@
         )
       )
-      (project "Quartz_v1p1"
+      (project "Quartz_v1p2"
         (path "/674e1e7f-67ba-4e85-a926-dcd5f6a22021/40baf21a-c5b6-4126-86f5-a663d00e8f52"
           (reference "C101") (unit 1)
