File: fmc.kicad_sch (KiCad schematic)
At the start: 6 parts, among them P1 ASP-134604-01, P2 ASP-134604-01

Commit message: Updated to version 1.2.1
This update fixes a few production documentation issues.
The boards will be functionally identical to v1.2.
With this update and going forward I moved away from version number as a part of filenames

Updates:
BOM ITEM 3 GRT155R61C474KE01D -> CGA2B3X7R1H473K050BB (wrong value)
BOM ITEM 7 GRM1885C1H101JA01D -> GRM1555C1H101JA01D (wrong size)

Corrected MPN description on BOM items 1&3 (CL05X105KP5NNNC &CL21A106KOQNNNE)

Updated Silkscreen with Version Number
Updated Schematic Title Block with current Date and Version Number
Other:
- company: (none) -> OspreyDCS
- title: (none) -> Quartz
Changed lines of the file:
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@@
 (kicad_sch (version 20230121) (generator eeschema)
   (paper "A3")
+  (title_block
+    (title "Quartz")
+    (date "2024-03-28")
+    (rev "v1.2.1")
+    (company "OspreyDCS")
+  )
   (junction (at 314.96 179.07) (diameter 0) (color 0 0 0 0)
   )
