File: Quartz.kicad_pcb (KiCad board)
At the start: 6 copper layers, 254 x 130 mm, 1233 parts, among them J1 DB37, J2 DB37, J4 Conn_02x10_Odd_Even, J5 PPS IN, J6 WP Jumper, K1001 EE2-12TNU-L, K101 EE2-12TNU-L, K1101 EE2-12TNU-L, K1201 EE2-12TNU-L, K1301 EE2-12TNU-L, K1401 EE2-12TNU-L, K1501 EE2-12TNU-L, K1601 EE2-12TNU-L, K1701 EE2-12TNU-L, K1801 EE2-12TNU-L, K1901 EE2-12TNU-L, K2001 EE2-12TNU-L, K201 EE2-12TNU-L, K2101 EE2-12TNU-L, K2201 EE2-12TNU-L, K2301 EE2-12TNU-L, K2401 EE2-12TNU-L, K2501 EE2-12TNU-L, K2601 EE2-12TNU-L, K2701 EE2-12TNU-L, K2801 EE2-12TNU-L, K2901 EE2-12TNU-L, K3001 EE2-12TNU-L, K301 EE2-12TNU-L, K3101 EE2-12TNU-L, K3201 EE2-12TNU-L, K401 EE2-12TNU-L, K501 EE2-12TNU-L, K601 EE2-12TNU-L, K701 EE2-12TNU-L, K801 EE2-12TNU-L, K901 EE2-12TNU-L, P1 ASP-134604-01, P2 ASP-134604-01, Q1 FDN335N, Q2 FDN335N, Q3 FDMC510P, U1 AD7768, U10 AD7768, U1001 INA851, U101 INA851, U11 ADR4540, U1101 INA851, U12 ADA4841-1, U1201 INA851, U13 AMC7823, U1301 INA851, U14 MAX4896, U1401 INA851, U15 MAX4896, U1501 INA851, U16 SI5330B-B00206-GM, U1601 INA851, U17 MAX4896, U1701 INA851, U18 MAX4896, U1801 INA851, U19 MAX4896, U1901 INA851, U2 ADR4540, U20 MAX4896, U2001 INA851, U201 INA851, U21 MAX4896, U2101 INA851, U2201 INA851, U23 MAX4896, U2301 INA851, U2401 INA851, U2501 INA851, U26 74AVC4T245, U2601 INA851, U27 AT24C64D, U2701 INA851, U2801 INA851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

Commit message: Updating design to cover reworks
Updating design to cover reworks.
This should now match what has been delivered to NASA GRE-ATF after the board reworks.
All outputs have been regenerated
Changes are:
1)Changed the clock splitter part to a 2.5V compatible part
2)Changed some caps on the MCLK lines to 0R resitors
Parts:
- R178: renamed from C178; value 100nF -> 0R
- R179: renamed from C179; value 100nF -> 0R
- R180: renamed from C180; value 100nF -> 0R
- R181: renamed from C181; value 100nF -> 0R
- R182: renamed from C182; value 100nF -> 0R
- R183: renamed from C183; value 100nF -> 0R
- R184: renamed from C184; value 100nF -> 0R
- R185: renamed from C185; value 100nF -> 0R
- TP11: value 12V -> ~
- U16: value SI5330B-B00206-GM -> SI5330B-B00205-GM
